Commit message: hw_int state: simulated motor rotation

File: urdf/cybergear_servo.urdf.xacro (robot description, xacro)
@@ -5,5 +5,5 @@
 -->
 <robot xmlns:xacro="http://www.ros.org/wiki/xacro" name="cybergear_servo">
-  <xacro:include filename="$(find cybergear_servo_description)/urdf/cybergear_servo.xacro"/>
+  <xacro:include filename="$(find quadro)/urdf/cybergear_servo.xacro"/>
   <link name="base_link">
   </link>

File: urdf/cybergear_servo.xacro (robot description, xacro)
@@ -14,5 +14,5 @@
       <visual>
         <geometry>
-          <mesh filename="package://cybergear_servo_description/meshes/cybergear_body.stl" scale="0.001 0.001 0.001"/>
+          <mesh filename="package://quadro/meshes/cybergear_body.stl" scale="0.001 0.001 0.001"/>
         </geometry>
       </visual>
@@ -41,5 +41,5 @@
         <origin rpy="0 0 0" xyz="0 0 -0.028"/>
         <geometry>
-          <mesh filename="package://cybergear_servo_description/meshes/cybergear_table.stl" scale="0.001 0.001 0.001"/>
+          <mesh filename="package://quadro/meshes/cybergear_table.stl" scale="0.001 0.001 0.001"/>
         </geometry>
       </visual>
@@ -57,5 +57,5 @@
       -->
     </link>
-    <ros2_control name="CybergearMotorWheelJoint" type="actuator">
+    <ros2_control name="CybergearActuators" type="actuator">
     <hardware>
       <plugin>quadro/CybergearActuator</plugin>

Commit message: dual motor works

File: urdf/cybergear_servo.urdf.xacro (robot description, xacro)
@@ -8,5 +8,5 @@
   <link name="base_link">
   </link>
-  <xacro:cybergear_servo name="demo" parent="base_link">
+  <xacro:cybergear_servo name="quadro" parent="base_link">
     <origin rpy="0 0 0" xyz="0 0 0.1"/>
   </xacro:cybergear_servo>

File: urdf/cybergear_servo.xacro (robot description, xacro)
@@ -6,10 +6,10 @@
 <robot xmlns:xacro="http://www.ros.org/wiki/xacro">
   <xacro:macro name="cybergear_servo" params="name parent *origin">
-    <joint name="${name}_base_joint" type="fixed">
-      <xacro:insert_block name="origin"/>
+    <joint name="${name}_FR1_base_joint" type="fixed">
+      <origin rpy="${-pi/2} 0 0" xyz="0.0 0 0.1"/>
       <parent link="${parent}"/>
-      <child link="${name}_cybergear_link"/>
+      <child link="${name}_FR1_link"/>
     </joint>
-    <link name="${name}_cybergear_link">
+    <link name="${name}_FR1_link">
       <visual>
         <geometry>
@@ -23,19 +23,13 @@
         </geometry>
       </collision>
-      <!-- TODO
-      <inertial>
-        <origin rpy="0 0 0" xyz="0 0 0"/>
-        <mass value="0.2528"/>
-      </inertial>
-      -->
     </link>
-    <joint name="cybergear" type="revolute">
+    <joint name="FR1" type="revolute">
       <origin rpy="0 0 0" xyz="0 0 0.028"/>
-      <parent link="${name}_cybergear_link"/>
-      <child link="${name}_cybergear_table_link"/>
+      <parent link="${name}_FR1_link"/>
+      <child link="${name}_FR1_table_link"/>
       <axis xyz="0 0 1"/>
       <limit effort="12" velocity="30" lower="-12.565" upper="12.565"/>
     </joint>
-    <link name="${name}_cybergear_table_link">
+    <link name="${name}_FR1_table_link">
       <visual>
         <origin rpy="0 0 0" xyz="0 0 -0.028"/>
@@ -50,10 +44,44 @@
         </geometry>
       </collision>
-      <!-- TODO
-      <inertial>
-        <origin rpy="0 0 0" xyz="0 0 0"/>
-        <mass value="0.0632"/>
-      </inertial>
-      -->
+    </link>
+    <!-- SECOND LINK -->
+    <joint name="${name}_FR2_base_joint" type="fixed">
+      <origin rpy="0 0 0" xyz="0.1 0 0.0"/>
+      <parent link="${parent}"/>
+      <child link="${name}_FR2_link"/>
+    </joint>
+    <link name="${name}_FR2_link">
+      <visual>
+        <geometry>
+          <mesh filename="package://quadro/meshes/cybergear_body.stl" scale="0.001 0.001 0.001"/>
+        </geometry>
+      </visual>
+      <collision>
+        <origin rpy="0 0 0" xyz="0 0 0.008"/>
+        <geometry>
+          <cylinder length="0.035" radius="0.042"/>
+        </geometry>
+      </collision>
+    </link>
+    <joint name="FR2" type="revolute">
+      <origin rpy="0 0 0" xyz="0 0 0.028"/>
+      <parent link="${name}_FR2_link"/>
+      <child link="${name}_FR2_table_link"/>
+      <axis xyz="0 0 1"/>
+      <limit effort="12" velocity="30" lower="-12.565" upper="12.565"/>
+    </joint>
+    <link name="${name}_FR2_table_link">
+      <visual>
+        <origin rpy="0 0 0" xyz="0 0 -0.028"/>
+        <geometry>
+          <mesh filename="package://quadro/meshes/cybergear_table.stl" scale="0.001 0.001 0.001"/>
+        </geometry>
+      </visual>
+      <collision>
+        <origin rpy="0 0 0" xyz="0 0 -0.005"/>
+        <geometry>
+          <cylinder length="0.01" radius="0.016"/>
+        </geometry>
+      </collision>
     </link>
     <ros2_control name="CybergearActuators" type="actuator">
@@ -80,5 +108,5 @@
       <param name="temperature_scale">0.1</param>
     </hardware>
-    <joint name="cybergear">
+    <joint name="FR1">
       <command_interface name="position">
       </command_interface>
@@ -86,10 +114,10 @@
       <state_interface name="velocity"/>
     </joint>
-    <!-- <joint name="cybergear2">
+    <joint name="FR2">
       <command_interface name="position">
       </command_interface>
       <state_interface name="position"/>
       <state_interface name="velocity"/>
-    </joint> -->
+    </joint>
   </ros2_control>
   </xacro:macro>
