Commit message: basic multi motor support added

File: urdf/cybergear_servo.xacro (robot description, xacro)
@@ -82,10 +82,14 @@
     <joint name="cybergear">
       <command_interface name="position">
-        <param name="min">-100</param>
-        <param name="max">100</param>
       </command_interface>
       <state_interface name="position"/>
       <state_interface name="velocity"/>
     </joint>
+    <!-- <joint name="cybergear2">
+      <command_interface name="position">
+      </command_interface>
+      <state_interface name="position"/>
+      <state_interface name="velocity"/>
+    </joint> -->
   </ros2_control>
   </xacro:macro>

Commit message: added auto zeroing

File: urdf/cybergear_servo.xacro (robot description, xacro)
@@ -7,5 +7,5 @@
   <xacro:macro name="cybergear_servo" params="name parent *origin">
     <joint name="${name}_FR1_base_joint" type="fixed">
-      <origin rpy="${-pi/2} 0 0" xyz="0.0 0 0.1"/>
+      <origin rpy="0 0 0" xyz="0.0 0.0 0.0"/>
       <parent link="${parent}"/>
       <child link="${name}_FR1_link"/>
@@ -47,5 +47,5 @@
     <!-- SECOND LINK -->
     <joint name="${name}_FR2_base_joint" type="fixed">
-      <origin rpy="0 0 0" xyz="0.1 0 0.0"/>
+      <origin rpy="0.0 0.0 0.0" xyz="0.0 0.0 0.05"/>
       <parent link="${parent}"/>
       <child link="${name}_FR2_link"/>
@@ -92,5 +92,5 @@
       <param name="use_bus_time">false</param>
       <param name="interval_sec">0.5</param>
-      <param name="device_id">127</param>
+      <param name="device_id">1</param>
       <param name="primary_id">0</param>
       <param name="max_position">12.56637061</param>

Commit message: streamlined creating messages

File: urdf/cybergear_servo.xacro (robot description, xacro)
@@ -47,6 +47,6 @@
     <!-- SECOND LINK -->
     <joint name="${name}_FR2_base_joint" type="fixed">
-      <origin rpy="0.0 0.0 0.0" xyz="0.0 0.0 0.05"/>
-      <parent link="${parent}"/>
+      <origin rpy="0.0 0.0 0.0" xyz="0.0 0.0 0.02"/>
+      <parent link="${name}_FR1_table_link"/>
       <child link="${name}_FR2_link"/>
     </joint>
@@ -92,19 +92,5 @@
       <param name="use_bus_time">false</param>
       <param name="interval_sec">0.5</param>
-      <param name="device_id">1</param>
       <param name="primary_id">0</param>
-      <param name="max_position">12.56637061</param>
-      <param name="min_position">-12.56637061</param>
-      <param name="max_velocity">30.0</param>
-      <param name="min_velocity">-30.0</param>
-      <param name="max_effort">12.0</param>
-      <param name="min_effort">-12.0</param>
-      <param name="max_gain_kp">500.0</param>
-      <param name="min_gain_kp">0.0</param>
-      <param name="max_gain_kd">5.0</param>
-      <param name="min_gain_kd">0.0</param>
-      <param name="max_current">23.0</param>
-      <param name="min_current">-23.0</param>
-      <param name="temperature_scale">0.1</param>
     </hardware>
     <joint name="FR1">
