Commit message: added second leg

File: description/leg.xacro (robot description, xacro)
@@ -19,7 +19,7 @@
   <link name="motor">
     <inertial>
-      <origin xyz="-0.0236869 0.0333936 0.0493711" rpy="0 0 0"/>
-      <mass value="0.586935"/>
-      <inertia ixx="0.000559915" ixy="9.50807e-06" ixz="0.000198772" iyy="0.00147041" iyz="-5.98234e-05" izz="0.0015943"/>
+      <origin xyz="0.000167595 0.0335997 0.0536899" rpy="0 0 0"/>
+      <mass value="0.840992"/>
+      <inertia ixx="0.000727199" ixy="-1.7348e-08" ixz="-1.37499e-06" iyy="0.00274647" iyz="-6.25483e-05" izz="0.00292446"/>
     </inertial>
     <!-- Part motor -->
@@ -69,4 +69,20 @@
       <geometry>
         <mesh filename="file://$(find quadro)/description/leg_assets/back_stop.stl"/>
+      </geometry>
+    </collision>
+    <!-- Part motor_2 -->
+    <visual>
+      <origin xyz="0.055 0.0342754 0.051" rpy="-1.5708 -1.5708 0"/>
+      <geometry>
+        <mesh filename="file://$(find quadro)/description/leg_assets/motor.stl"/>
+      </geometry>
+      <material name="motor_2_material">
+        <color rgba="0.498039 0.498039 0.498039 1"/>
+      </material>
+    </visual>
+    <collision>
+      <origin xyz="0.055 0.0342754 0.051" rpy="-1.5708 -1.5708 0"/>
+      <geometry>
+        <mesh filename="file://$(find quadro)/description/leg_assets/motor.stl"/>
       </geometry>
     </collision>
@@ -111,5 +127,5 @@
       </geometry>
     </collision>
-    <!-- Part motor_2 -->
+    <!-- Part motor_3 -->
     <visual>
       <origin xyz="-0.0085 -0.0147224 -0.0735" rpy="-1.5708 1.52638e-15 1.0472"/>
@@ -117,5 +133,5 @@
         <mesh filename="file://$(find quadro)/description/leg_assets/motor.stl"/>
       </geometry>
-      <material name="motor_2_material">
+      <material name="motor_3_material">
         <color rgba="0.498039 0.498039 0.498039 1"/>
       </material>
@@ -137,5 +153,5 @@
     <!-- Part lin_2_br -->
     <visual>
-      <origin xyz="-0.0577297 0.123802 -0.0195" rpy="1.5708 6.50343e-15 2.00713"/>
+      <origin xyz="-0.0577297 0.123802 -0.0195" rpy="1.5708 1.94085e-14 2.00713"/>
       <geometry>
         <mesh filename="file://$(find quadro)/description/leg_assets/lin_2_br.stl"/>
@@ -146,5 +162,5 @@
     </visual>
     <collision>
-      <origin xyz="-0.0577297 0.123802 -0.0195" rpy="1.5708 6.50343e-15 2.00713"/>
+      <origin xyz="-0.0577297 0.123802 -0.0195" rpy="1.5708 1.94085e-14 2.00713"/>
       <geometry>
         <mesh filename="file://$(find quadro)/description/leg_assets/lin_2_br.stl"/>
@@ -153,5 +169,5 @@
     <!-- Part shaft_2 -->
     <visual>
-      <origin xyz="1.38778e-17 2.77556e-17 0.01" rpy="1.5708 1.5708 0"/>
+      <origin xyz="1.38778e-17 0 0.01" rpy="1.5708 1.5708 0"/>
       <geometry>
         <mesh filename="file://$(find quadro)/description/leg_assets/shaft.stl"/>
@@ -162,5 +178,5 @@
     </visual>
     <collision>
-      <origin xyz="1.38778e-17 2.77556e-17 0.01" rpy="1.5708 1.5708 0"/>
+      <origin xyz="1.38778e-17 0 0.01" rpy="1.5708 1.5708 0"/>
       <geometry>
         <mesh filename="file://$(find quadro)/description/leg_assets/shaft.stl"/>
@@ -169,5 +185,5 @@
     <!-- Part lin_3_top_r -->
     <visual>
-      <origin xyz="8.11851e-16 -1.38778e-16 -0.0645" rpy="1.5708 -4.26631e-15 1.22173"/>
+      <origin xyz="7.91034e-16 -1.11022e-16 -0.0645" rpy="1.5708 -1.25557e-14 1.22173"/>
       <geometry>
         <mesh filename="file://$(find quadro)/description/leg_assets/lin_3_top_r.stl"/>
@@ -178,5 +194,5 @@
     </visual>
     <collision>
-      <origin xyz="8.11851e-16 -1.38778e-16 -0.0645" rpy="1.5708 -4.26631e-15 1.22173"/>
+      <origin xyz="7.91034e-16 -1.11022e-16 -0.0645" rpy="1.5708 -1.25557e-14 1.22173"/>
       <geometry>
         <mesh filename="file://$(find quadro)/description/leg_assets/lin_3_top_r.stl"/>
@@ -185,5 +201,5 @@
     <!-- Part lin_3_bot_r -->
     <visual>
-      <origin xyz="8.32667e-16 -2.77556e-17 -0.0645" rpy="1.5708 -4.18305e-15 1.22173"/>
+      <origin xyz="8.18789e-16 0 -0.0645" rpy="1.5708 -1.25835e-14 1.22173"/>
       <geometry>
         <mesh filename="file://$(find quadro)/description/leg_assets/lin_3_bot_r.stl"/>
@@ -194,21 +210,21 @@
     </visual>
     <collision>
-      <origin xyz="8.32667e-16 -2.77556e-17 -0.0645" rpy="1.5708 -4.18305e-15 1.22173"/>
+      <origin xyz="8.18789e-16 0 -0.0645" rpy="1.5708 -1.25835e-14 1.22173"/>
       <geometry>
         <mesh filename="file://$(find quadro)/description/leg_assets/lin_3_bot_r.stl"/>
       </geometry>
     </collision>
-    <!-- Part motor_3 -->
-    <visual>
-      <origin xyz="8.39606e-16 -5.55112e-17 -0.0385" rpy="2.70526 1.5708 0"/>
-      <geometry>
-        <mesh filename="file://$(find quadro)/description/leg_assets/motor.stl"/>
-      </geometry>
-      <material name="motor_3_material">
-        <color rgba="0.498039 0.498039 0.498039 1"/>
-      </material>
-    </visual>
-    <collision>
-      <origin xyz="8.39606e-16 -5.55112e-17 -0.0385" rpy="2.70526 1.5708 0"/>
+    <!-- Part motor_4 -->
+    <visual>
+      <origin xyz="8.25728e-16 -2.77556e-17 -0.0385" rpy="2.70526 1.5708 0"/>
+      <geometry>
+        <mesh filename="file://$(find quadro)/description/leg_assets/motor.stl"/>
+      </geometry>
+      <material name="motor_4_material">
+        <color rgba="0.498039 0.498039 0.498039 1"/>
+      </material>
+    </visual>
+    <collision>
+      <origin xyz="8.25728e-16 -2.77556e-17 -0.0385" rpy="2.70526 1.5708 0"/>
       <geometry>
         <mesh filename="file://$(find quadro)/description/leg_assets/motor.stl"/>
@@ -217,5 +233,5 @@
     <!-- Part bearing -->
     <visual>
-      <origin xyz="-0.068404 -0.187939 -0.074" rpy="3.14159 -1.23311e-14 0.436332"/>
+      <origin xyz="-0.068404 -0.187939 -0.074" rpy="3.14159 -3.7582e-14 0.436332"/>
       <geometry>
         <mesh filename="file://$(find quadro)/description/leg_assets/bearing.stl"/>
@@ -226,5 +242,5 @@
     </visual>
     <collision>
-      <origin xyz="-0.068404 -0.187939 -0.074" rpy="3.14159 -1.23311e-14 0.436332"/>
+      <origin xyz="-0.068404 -0.187939 -0.074" rpy="3.14159 -3.7582e-14 0.436332"/>
       <geometry>
         <mesh filename="file://$(find quadro)/description/leg_assets/bearing.stl"/>
@@ -241,5 +257,5 @@
     <!-- Part lin_top_r -->
     <visual>
-      <origin xyz="-2.77556e-17 -2.77556e-17 0.003" rpy="1.5708 1.99014e-16 0"/>
+      <origin xyz="-2.77556e-17 4.16334e-17 0.003" rpy="1.5708 -7.50078e-16 5.55112e-17"/>
       <geometry>
         <mesh filename="file://$(find quadro)/description/leg_assets/lin_top_r.stl"/>
@@ -250,5 +266,5 @@
     </visual>
     <collision>
-      <origin xyz="-2.77556e-17 -2.77556e-17 0.003" rpy="1.5708 1.99014e-16 0"/>
+      <origin xyz="-2.77556e-17 4.16334e-17 0.003" rpy="1.5708 -7.50078e-16 5.55112e-17"/>
       <geometry>
         <mesh filename="file://$(find quadro)/description/leg_assets/lin_top_r.stl"/>
@@ -257,5 +273,5 @@
     <!-- Part bearing_2 -->
     <visual>
-      <origin xyz="-4.16334e-17 -0.05 -0.0255" rpy="3.14159 8.79922e-17 -1.66533e-16"/>
+      <origin xyz="0 -0.05 -0.0255" rpy="-3.14159 -1.19417e-15 -5.55112e-17"/>
       <geometry>
         <mesh filename="file://$(find quadro)/description/leg_assets/bearing.stl"/>
@@ -266,5 +282,5 @@
     </visual>
     <collision>
-      <origin xyz="-4.16334e-17 -0.05 -0.0255" rpy="3.14159 8.79922e-17 -1.66533e-16"/>
+      <origin xyz="0 -0.05 -0.0255" rpy="-3.14159 -1.19417e-15 -5.55112e-17"/>
       <geometry>
         <mesh filename="file://$(find quadro)/description/leg_assets/bearing.stl"/>
@@ -273,5 +289,5 @@
     <!-- Part shaft_3 -->
     <visual>
-      <origin xyz="-1.38778e-17 -1.38778e-17 0.01" rpy="1.5708 1.5708 0"/>
+      <origin xyz="0 1.38778e-17 0.01" rpy="1.5708 1.5708 0"/>
       <geometry>
         <mesh filename="file://$(find quadro)/description/leg_assets/shaft.stl"/>
@@ -282,5 +298,5 @@
     </visual>
     <collision>
-      <origin xyz="-1.38778e-17 -1.38778e-17 0.01" rpy="1.5708 1.5708 0"/>
+      <origin xyz="0 1.38778e-17 0.01" rpy="1.5708 1.5708 0"/>
       <geometry>
         <mesh filename="file://$(find quadro)/description/leg_assets/shaft.stl"/>
@@ -290,10 +306,9 @@
   <!-- Joint from lin_2_br to lin_top_r -->
   <joint name="joint_br_3" type="revolute">
-    <origin xyz="8.46545e-16 -2.77556e-17 -0.0485" rpy="-5.42096e-15 -1.33858e-14 0.436332"/>
+    <origin xyz="8.25728e-16 -8.32667e-17 -0.0485" rpy="-1.90199e-14 -3.69158e-14 0.436332"/>
     <parent link="lin_2_br"/>
     <child link="lin_top_r"/>
     <axis xyz="0 0 -1"/>
-    <limit effort="10" velocity="12" lower="-3.14" upper="3.14"/>
-    <joint_properties friction="0.5"/>
+    <limit effort="10" velocity="10" lower="-3.141592653589793" upper="3.141592653589793"/>
   </joint>
   <!-- Link lin_4_r -->
@@ -306,5 +321,5 @@
     <!-- Part lin_4_r -->
     <visual>
-      <origin xyz="0.2 -6.91114e-15 -0.0085" rpy="-1.5708 -1.96624e-17 -3.4972e-14"/>
+      <origin xyz="0.2 -7.88258e-15 -0.0085" rpy="-1.5708 -1.18604e-16 -3.9746e-14"/>
       <geometry>
         <mesh filename="file://$(find quadro)/description/leg_assets/lin_4_r.stl"/>
@@ -315,5 +330,5 @@
     </visual>
     <collision>
-      <origin xyz="0.2 -6.91114e-15 -0.0085" rpy="-1.5708 -1.96624e-17 -3.4972e-14"/>
+      <origin xyz="0.2 -7.88258e-15 -0.0085" rpy="-1.5708 -1.18604e-16 -3.9746e-14"/>
       <geometry>
         <mesh filename="file://$(find quadro)/description/leg_assets/lin_4_r.stl"/>
@@ -322,5 +337,5 @@
     <!-- Part bearing_3 -->
     <visual>
-      <origin xyz="1.72085e-15 0.05 -1.38778e-17" rpy="3.14159 -1.96624e-17 -3.49165e-14"/>
+      <origin xyz="1.94289e-15 0.05 -1.38778e-17" rpy="3.14159 -1.18604e-16 -3.95795e-14"/>
       <geometry>
         <mesh filename="file://$(find quadro)/description/leg_assets/bearing.stl"/>
@@ -331,5 +346,5 @@
     </visual>
     <collision>
-      <origin xyz="1.72085e-15 0.05 -1.38778e-17" rpy="3.14159 -1.96624e-17 -3.49165e-14"/>
+      <origin xyz="1.94289e-15 0.05 -1.38778e-17" rpy="3.14159 -1.18604e-16 -3.95795e-14"/>
       <geometry>
         <mesh filename="file://$(find quadro)/description/leg_assets/bearing.stl"/>
@@ -338,21 +353,19 @@
   </link>
   <!-- Joint from lin_2_br to lin_4_r -->
-  <joint name="l4_l3" type="revolute">
-    <origin xyz="-0.068404 -0.187939 -0.074" rpy="3.14159 -1.23311e-14 0.436332"/>
+  <joint name="br_l4_l3" type="revolute">
+    <origin xyz="-0.068404 -0.187939 -0.074" rpy="3.14159 -3.7582e-14 0.436332"/>
     <parent link="lin_2_br"/>
     <child link="lin_4_r"/>
     <axis xyz="0 0 -1"/>
-    <limit effort="10" velocity="12" lower="-3.14" upper="3.14"/>
-    <joint_properties friction="0.5"/>
+    <limit effort="10" velocity="10" lower="-3.141592653589793" upper="3.141592653589793"/>
     <mimic joint="joint_br_3" multiplier="-1.0"/>
   </joint>
   <!-- Joint from shaft to lin_2_br -->
   <joint name="joint_br_2" type="revolute">
-    <origin xyz="-0.0035 -0.00606218 -0.0735" rpy="1.5708 -0.0310412 -0.523599"/>
+    <origin xyz="-0.0035 -0.00606218 -0.0735" rpy="1.5708 8.1119e-15 -0.523599"/>
     <parent link="shaft"/>
     <child link="lin_2_br"/>
     <axis xyz="0 0 -1"/>
-    <limit effort="10" velocity="12" lower="-3.14" upper="3.14"/>
-    <joint_properties friction="0.5"/>
+    <limit effort="10" velocity="10" lower="-3.141592653589793" upper="3.141592653589793"/>
   </joint>
   <!-- Joint from motor to shaft -->
@@ -362,6 +375,294 @@
     <child link="shaft"/>
     <axis xyz="0 0 -1"/>
-    <limit effort="10" velocity="12" lower="-3.14" upper="3.14"/>
-    <joint_properties friction="0.5"/>
+    <limit effort="10" velocity="10" lower="-3.141592653589793" upper="3.141592653589793"/>
+  </joint>
+  <!-- Link shaft_2 -->
+  <link name="shaft_2">
+    <inertial>
+      <origin xyz="-0.00365203 0.00743033 -0.0535667" rpy="0 0 0"/>
+      <mass value="0.500834"/>
+      <inertia ixx="0.000662397" ixy="-4.87254e-05" ixz="-1.77194e-05" iyy="0.000709837" iyz="3.40867e-05" izz="0.000280763"/>
+    </inertial>
+    <!-- Part shaft_4 -->
+    <visual>
+      <origin xyz="0 0 0.01" rpy="1.5708 1.5708 0"/>
+      <geometry>
+        <mesh filename="file://$(find quadro)/description/leg_assets/shaft.stl"/>
+      </geometry>
+      <material name="shaft_4_material">
+        <color rgba="0.498039 0.498039 0.498039 1"/>
+      </material>
+    </visual>
+    <collision>
+      <origin xyz="0 0 0.01" rpy="1.5708 1.5708 0"/>
+      <geometry>
+        <mesh filename="file://$(find quadro)/description/leg_assets/shaft.stl"/>
+      </geometry>
+    </collision>
+    <!-- Part motor_5 -->
+    <visual>
+      <origin xyz="-0.0085 0.0147224 -0.0735" rpy="1.5708 8.92383e-17 -1.0472"/>
+      <geometry>
+        <mesh filename="file://$(find quadro)/description/leg_assets/motor.stl"/>
+      </geometry>
+      <material name="motor_5_material">
+        <color rgba="0.498039 0.498039 0.498039 1"/>
+      </material>
+    </visual>
+    <collision>
+      <origin xyz="-0.0085 0.0147224 -0.0735" rpy="1.5708 8.92383e-17 -1.0472"/>
+      <geometry>
+        <mesh filename="file://$(find quadro)/description/leg_assets/motor.stl"/>
+      </geometry>
+    </collision>
+    <!-- Part lin_1_support_bl -->
+    <visual>
+      <origin xyz="-0.0485 0.0840045 -0.0735" rpy="-2.61799 -1.5708 0"/>
+      <geometry>
+        <mesh filename="file://$(find quadro)/description/leg_assets/lin_1_support_bl.stl"/>
+      </geometry>
+      <material name="lin_1_support_bl_material">
+        <color rgba="1 0.756863 0.054902 1"/>
+      </material>
+    </visual>
+    <collision>
+      <origin xyz="-0.0485 0.0840045 -0.0735" rpy="-2.61799 -1.5708 0"/>
+      <geometry>
+        <mesh filename="file://$(find quadro)/description/leg_assets/lin_1_support_bl.stl"/>
+      </geometry>
+    </collision>
+  </link>
+  <!-- Link motor_2 -->
+  <link name="motor_2">
+    <inertial>
+      <origin xyz="-0.00512367 0.0104232 -0.0435875" rpy="0 0 0"/>
+      <mass value="0.551476"/>
+      <inertia ixx="0.00130661" ixy="0.000304518" ixz="-9.96006e-05" iyy="0.000599134" iyz="0.000185395" izz="0.00132552"/>
+    </inertial>
+    <!-- Part lin_3_top_l -->
+    <visual>
+      <origin xyz="6.52256e-16 1.11022e-16 0.087" rpy="-1.5708 7.28298e-16 -1.22173"/>
+      <geometry>
+        <mesh filename="file://$(find quadro)/description/leg_assets/lin_3_top_l.stl"/>
+      </geometry>
+      <material name="lin_3_top_l_material">
+        <color rgba="1 0.756863 0.054902 1"/>
+      </material>
+    </visual>
+    <collision>
+      <origin xyz="6.52256e-16 1.11022e-16 0.087" rpy="-1.5708 7.28298e-16 -1.22173"/>
+      <geometry>
+        <mesh filename="file://$(find quadro)/description/leg_assets/lin_3_top_l.stl"/>
+      </geometry>
+    </collision>
+    <!-- Part lin_2_bl -->
+    <visual>
+      <origin xyz="-6.93889e-18 -5.55112e-17 -0.0195" rpy="1.5708 4.12056e-17 1.13446"/>
+      <geometry>
+        <mesh filename="file://$(find quadro)/description/leg_assets/lin_2_bl.stl"/>
+      </geometry>
+      <material name="lin_2_bl_material">
+        <color rgba="1 0.756863 0.054902 1"/>
+      </material>
+    </visual>
+    <collision>
+      <origin xyz="-6.93889e-18 -5.55112e-17 -0.0195" rpy="1.5708 4.12056e-17 1.13446"/>
+      <geometry>
+        <mesh filename="file://$(find quadro)/description/leg_assets/lin_2_bl.stl"/>
+      </geometry>
+    </collision>
+    <!-- Part lin_3_bot_l -->
+    <visual>
+      <origin xyz="6.80012e-16 5.55112e-17 0.087" rpy="-1.5708 -4.65192e-16 -1.22173"/>
+      <geometry>
+        <mesh filename="file://$(find quadro)/description/leg_assets/lin_3_bot_l.stl"/>
+      </geometry>
+      <material name="lin_3_bot_l_material">
+        <color rgba="1 0.756863 0.054902 1"/>
+      </material>
+    </visual>
+    <collision>
+      <origin xyz="6.80012e-16 5.55112e-17 0.087" rpy="-1.5708 -4.65192e-16 -1.22173"/>
+      <geometry>
+        <mesh filename="file://$(find quadro)/description/leg_assets/lin_3_bot_l.stl"/>
+      </geometry>
+    </collision>
+    <!-- Part shaft_5 -->
+    <visual>
+      <origin xyz="0 0 0.01" rpy="1.5708 1.5708 0"/>
+      <geometry>
+        <mesh filename="file://$(find quadro)/description/leg_assets/shaft.stl"/>
+      </geometry>
+      <material name="shaft_5_material">
+        <color rgba="0.498039 0.498039 0.498039 1"/>
+      </material>
+    </visual>
+    <collision>
+      <origin xyz="0 0 0.01" rpy="1.5708 1.5708 0"/>
+      <geometry>
+        <mesh filename="file://$(find quadro)/description/leg_assets/shaft.stl"/>
+      </geometry>
+    </collision>
+    <!-- Part motor_6 -->
+    <visual>
+      <origin xyz="8.95117e-16 2.77556e-17 -0.0385" rpy="-2.70526 1.5708 0"/>
+      <geometry>
+        <mesh filename="file://$(find quadro)/description/leg_assets/motor.stl"/>
+      </geometry>
+      <material name="motor_6_material">
+        <color rgba="0.498039 0.498039 0.498039 1"/>
+      </material>
+    </visual>
+    <collision>
+      <origin xyz="8.95117e-16 2.77556e-17 -0.0385" rpy="-2.70526 1.5708 0"/>
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