Commit message: onto something with back legs

File: description/leg_rotated.xacro (robot description, xacro)
@@ -16,4 +16,5 @@
     <child link="motor"/>
   </joint>
+  <!-- Link motor -->
   <link name="motor">
     <inertial>
@@ -90,11 +91,11 @@
   <link name="shaft">
     <inertial>
-      <origin xyz="0.000552419 -0.00826087 -0.0538481" rpy="0 0 0"/>
+      <origin xyz="-0.00365203 -0.00743033 -0.0538481" rpy="0 0 0"/>
       <mass value="0.500834"/>
-      <inertia ixx="0.000637639" ixy="3.82058e-06" ixz="1.69793e-06" iyy="0.000745753" iyz="-3.78573e-05" izz="0.000280763"/>
+      <inertia ixx="0.000667976" ixy="4.87254e-05" ixz="-1.74582e-05" iyy="0.000715416" iyz="-3.36343e-05" izz="0.000280763"/>
     </inertial>
     <!-- Part lin_1_support_br -->
     <visual>
-      <origin xyz="-6.93889e-18 -0.028 -0.0735" rpy="-3.14159 -1.5708 0"/>
+      <origin xyz="-0.014 -0.0242487 -0.0735" rpy="2.61799 -1.5708 0"/>
       <geometry>
         <mesh filename="file://$(find quadro)/description/leg_assets/lin_1_support_br.stl"/>
@@ -105,5 +106,5 @@
     </visual>
     <collision>
-      <origin xyz="-6.93889e-18 -0.028 -0.0735" rpy="-3.14159 -1.5708 0"/>
+      <origin xyz="-0.014 -0.0242487 -0.0735" rpy="2.61799 -1.5708 0"/>
       <geometry>
         <mesh filename="file://$(find quadro)/description/leg_assets/lin_1_support_br.stl"/>
@@ -112,5 +113,5 @@
     <!-- Part shaft -->
     <visual>
-      <origin xyz="-6.93889e-18 0 0.01" rpy="1.5708 1.5708 0"/>
+      <origin xyz="0 0 0.01" rpy="1.5708 1.5708 0"/>
       <geometry>
         <mesh filename="file://$(find quadro)/description/leg_assets/shaft.stl"/>
@@ -121,5 +122,5 @@
     </visual>
     <collision>
-      <origin xyz="-6.93889e-18 0 0.01" rpy="1.5708 1.5708 0"/>
+      <origin xyz="0 0 0.01" rpy="1.5708 1.5708 0"/>
       <geometry>
         <mesh filename="file://$(find quadro)/description/leg_assets/shaft.stl"/>
@@ -128,5 +129,5 @@
     <!-- Part motor_3 -->
     <visual>
-      <origin xyz="-2.77556e-17 -0.017 -0.0735" rpy="-1.5708 2.17963e-16 1.5708"/>
+      <origin xyz="-0.0085 -0.0147224 -0.0735" rpy="-1.5708 1.52638e-15 1.0472"/>
       <geometry>
         <mesh filename="file://$(find quadro)/description/leg_assets/motor.stl"/>
@@ -137,5 +138,5 @@
     </visual>
     <collision>
-      <origin xyz="-2.77556e-17 -0.017 -0.0735" rpy="-1.5708 2.17963e-16 1.5708"/>
+      <origin xyz="-0.0085 -0.0147224 -0.0735" rpy="-1.5708 1.52638e-15 1.0472"/>
       <geometry>
         <mesh filename="file://$(find quadro)/description/leg_assets/motor.stl"/>
@@ -152,5 +153,5 @@
     <!-- Part lin_2_br -->
     <visual>
-      <origin xyz="-0.0577297 0.123802 -0.0195" rpy="1.5708 -4.403e-17 2.00713"/>
+      <origin xyz="-0.0577297 0.123802 -0.0195" rpy="1.5708 1.94085e-14 2.00713"/>
       <geometry>
         <mesh filename="file://$(find quadro)/description/leg_assets/lin_2_br.stl"/>
@@ -161,5 +162,5 @@
     </visual>
     <collision>
-      <origin xyz="-0.0577297 0.123802 -0.0195" rpy="1.5708 -4.403e-17 2.00713"/>
+      <origin xyz="-0.0577297 0.123802 -0.0195" rpy="1.5708 1.94085e-14 2.00713"/>
       <geometry>
         <mesh filename="file://$(find quadro)/description/leg_assets/lin_2_br.stl"/>
@@ -168,5 +169,5 @@
     <!-- Part shaft_2 -->
     <visual>
-      <origin xyz="0 0 0.01" rpy="1.5708 1.5708 0"/>
+      <origin xyz="1.38778e-17 0 0.01" rpy="1.5708 1.5708 0"/>
       <geometry>
         <mesh filename="file://$(find quadro)/description/leg_assets/shaft.stl"/>
@@ -177,5 +178,5 @@
     </visual>
     <collision>
-      <origin xyz="0 0 0.01" rpy="1.5708 1.5708 0"/>
+      <origin xyz="1.38778e-17 0 0.01" rpy="1.5708 1.5708 0"/>
       <geometry>
         <mesh filename="file://$(find quadro)/description/leg_assets/shaft.stl"/>
@@ -184,5 +185,5 @@
     <!-- Part lin_3_top_r -->
     <visual>
-      <origin xyz="7.97973e-16 -1.94289e-16 -0.0645" rpy="1.5708 1.70749e-16 1.22173"/>
+      <origin xyz="7.91034e-16 -1.11022e-16 -0.0645" rpy="1.5708 -1.25557e-14 1.22173"/>
       <geometry>
         <mesh filename="file://$(find quadro)/description/leg_assets/lin_3_top_r.stl"/>
@@ -193,5 +194,5 @@
     </visual>
     <collision>
-      <origin xyz="7.97973e-16 -1.94289e-16 -0.0645" rpy="1.5708 1.70749e-16 1.22173"/>
+      <origin xyz="7.91034e-16 -1.11022e-16 -0.0645" rpy="1.5708 -1.25557e-14 1.22173"/>
       <geometry>
         <mesh filename="file://$(find quadro)/description/leg_assets/lin_3_top_r.stl"/>
@@ -200,5 +201,5 @@
     <!-- Part lin_3_bot_r -->
     <visual>
-      <origin xyz="8.18789e-16 -1.11022e-16 -0.0645" rpy="1.5708 -2.28168e-17 1.22173"/>
+      <origin xyz="8.18789e-16 0 -0.0645" rpy="1.5708 -1.25835e-14 1.22173"/>
       <geometry>
         <mesh filename="file://$(find quadro)/description/leg_assets/lin_3_bot_r.stl"/>
@@ -209,5 +210,5 @@
     </visual>
     <collision>
-      <origin xyz="8.18789e-16 -1.11022e-16 -0.0645" rpy="1.5708 -2.28168e-17 1.22173"/>
+      <origin xyz="8.18789e-16 0 -0.0645" rpy="1.5708 -1.25835e-14 1.22173"/>
       <geometry>
         <mesh filename="file://$(find quadro)/description/leg_assets/lin_3_bot_r.stl"/>
@@ -216,5 +217,5 @@
     <!-- Part motor_4 -->
     <visual>
-      <origin xyz="8.18789e-16 -1.11022e-16 -0.0385" rpy="2.70526 1.5708 0"/>
+      <origin xyz="8.25728e-16 -2.77556e-17 -0.0385" rpy="2.70526 1.5708 0"/>
       <geometry>
         <mesh filename="file://$(find quadro)/description/leg_assets/motor.stl"/>
@@ -225,5 +226,5 @@
     </visual>
     <collision>
-      <origin xyz="8.18789e-16 -1.11022e-16 -0.0385" rpy="2.70526 1.5708 0"/>
+      <origin xyz="8.25728e-16 -2.77556e-17 -0.0385" rpy="2.70526 1.5708 0"/>
       <geometry>
         <mesh filename="file://$(find quadro)/description/leg_assets/motor.stl"/>
@@ -232,5 +233,5 @@
     <!-- Part bearing -->
     <visual>
-      <origin xyz="-0.068404 -0.187939 -0.074" rpy="-3.14159 -1.01626e-15 0.436332"/>
+      <origin xyz="-0.068404 -0.187939 -0.074" rpy="3.14159 -3.7582e-14 0.436332"/>
       <geometry>
         <mesh filename="file://$(find quadro)/description/leg_assets/bearing.stl"/>
@@ -241,5 +242,5 @@
     </visual>
     <collision>
-      <origin xyz="-0.068404 -0.187939 -0.074" rpy="-3.14159 -1.01626e-15 0.436332"/>
+      <origin xyz="-0.068404 -0.187939 -0.074" rpy="3.14159 -3.7582e-14 0.436332"/>
       <geometry>
         <mesh filename="file://$(find quadro)/description/leg_assets/bearing.stl"/>
@@ -256,5 +257,5 @@
     <!-- Part lin_top_r -->
     <visual>
-      <origin xyz="-2.77556e-17 -2.77556e-17 0.003" rpy="1.5708 8.71885e-16 1.11022e-16"/>
+      <origin xyz="-2.77556e-17 4.16334e-17 0.003" rpy="1.5708 -7.50078e-16 5.55112e-17"/>
       <geometry>
         <mesh filename="file://$(find quadro)/description/leg_assets/lin_top_r.stl"/>
@@ -265,5 +266,5 @@
     </visual>
     <collision>
-      <origin xyz="-2.77556e-17 -2.77556e-17 0.003" rpy="1.5708 8.71885e-16 1.11022e-16"/>
+      <origin xyz="-2.77556e-17 4.16334e-17 0.003" rpy="1.5708 -7.50078e-16 5.55112e-17"/>
       <geometry>
         <mesh filename="file://$(find quadro)/description/leg_assets/lin_top_r.stl"/>
@@ -272,5 +273,5 @@
     <!-- Part bearing_2 -->
     <visual>
-      <origin xyz="0 -0.05 -0.0255" rpy="3.14159 -1.52333e-15 1.11022e-16"/>
+      <origin xyz="0 -0.05 -0.0255" rpy="-3.14159 -1.19417e-15 -5.55112e-17"/>
       <geometry>
         <mesh filename="file://$(find quadro)/description/leg_assets/bearing.stl"/>
@@ -281,5 +282,5 @@
     </visual>
     <collision>
-      <origin xyz="0 -0.05 -0.0255" rpy="3.14159 -1.52333e-15 1.11022e-16"/>
+      <origin xyz="0 -0.05 -0.0255" rpy="-3.14159 -1.19417e-15 -5.55112e-17"/>
       <geometry>
         <mesh filename="file://$(find quadro)/description/leg_assets/bearing.stl"/>
@@ -288,5 +289,5 @@
     <!-- Part shaft_3 -->
     <visual>
-      <origin xyz="-2.77556e-17 -1.38778e-17 0.01" rpy="1.5708 1.5708 0"/>
+      <origin xyz="0 1.38778e-17 0.01" rpy="1.5708 1.5708 0"/>
       <geometry>
         <mesh filename="file://$(find quadro)/description/leg_assets/shaft.stl"/>
@@ -297,5 +298,5 @@
     </visual>
     <collision>
-      <origin xyz="-2.77556e-17 -1.38778e-17 0.01" rpy="1.5708 1.5708 0"/>
+      <origin xyz="0 1.38778e-17 0.01" rpy="1.5708 1.5708 0"/>
       <geometry>
         <mesh filename="file://$(find quadro)/description/leg_assets/shaft.stl"/>
@@ -305,9 +306,9 @@
   <!-- Joint from lin_2_br to lin_top_r -->
   <joint name="joint_br_3" type="revolute">
-    <origin xyz="8.18789e-16 -8.32667e-17 -0.0485" rpy="1.70478e-15 -9.46644e-17 0.436332"/>
+    <origin xyz="8.25728e-16 -8.32667e-17 -0.0485" rpy="-1.90199e-14 -3.69158e-14 0.436332"/>
     <parent link="lin_2_br"/>
     <child link="lin_top_r"/>
     <axis xyz="0 0 -1"/>
-    <limit effort="10" velocity="10" lower="-6.281592653589793" upper="6.281592653589793"/>
+    <limit effort="10" velocity="10" lower="-3.141592653589793" upper="3.141592653589793"/>
   </joint>
   <!-- Link lin_4_r -->
@@ -320,5 +321,5 @@
     <!-- Part lin_4_r -->
     <visual>
-      <origin xyz="0.2 -4.02456e-15 -0.0085" rpy="-1.5708 1.90985e-18 -2.03171e-14"/>
+      <origin xyz="0.2 -7.88258e-15 -0.0085" rpy="-1.5708 -1.18604e-16 -3.9746e-14"/>
       <geometry>
         <mesh filename="file://$(find quadro)/description/leg_assets/lin_4_r.stl"/>
@@ -329,5 +330,5 @@
     </visual>
     <collision>
-      <origin xyz="0.2 -4.02456e-15 -0.0085" rpy="-1.5708 1.90985e-18 -2.03171e-14"/>
+      <origin xyz="0.2 -7.88258e-15 -0.0085" rpy="-1.5708 -1.18604e-16 -3.9746e-14"/>
       <geometry>
         <mesh filename="file://$(find quadro)/description/leg_assets/lin_4_r.stl"/>
@@ -336,5 +337,5 @@
     <!-- Part bearing_3 -->
     <visual>
-      <origin xyz="8.88178e-16 0.05 -4.16334e-17" rpy="3.14159 4.78908e-17 -2.00395e-14"/>
+      <origin xyz="1.94289e-15 0.05 -1.38778e-17" rpy="3.14159 -1.18604e-16 -3.95795e-14"/>
       <geometry>
         <mesh filename="file://$(find quadro)/description/leg_assets/bearing.stl"/>
@@ -345,5 +346,5 @@
     </visual>
     <collision>
-      <origin xyz="8.88178e-16 0.05 -4.16334e-17" rpy="3.14159 4.78908e-17 -2.00395e-14"/>
+      <origin xyz="1.94289e-15 0.05 -1.38778e-17" rpy="3.14159 -1.18604e-16 -3.95795e-14"/>
       <geometry>
         <mesh filename="file://$(find quadro)/description/leg_assets/bearing.stl"/>
@@ -353,33 +354,33 @@
   <!-- Joint from lin_2_br to lin_4_r -->
   <joint name="br_l4_l3" type="revolute">
-    <origin xyz="-0.068404 -0.187939 -0.074" rpy="-3.14159 -1.01626e-15 0.436332"/>
+    <origin xyz="-0.068404 -0.187939 -0.074" rpy="3.14159 -3.7582e-14 0.436332"/>
     <parent link="lin_2_br"/>
     <child link="lin_4_r"/>
     <axis xyz="0 0 -1"/>
-    <limit effort="10" velocity="10" lower="-6.281592653589793" upper="6.281592653589793"/>
+    <limit effort="10" velocity="10" lower="-3.141592653589793" upper="3.141592653589793"/>
     <mimic joint="joint_br_3" multiplier="-1.0"/>
   </joint>
   <!-- Joint from shaft to lin_2_br -->
   <joint name="joint_br_2" type="revolute">
-    <origin xyz="-2.77556e-17 -0.007 -0.0735" rpy="1.5708 4.05346e-15 4.12283e-16"/>
+    <origin xyz="-0.0035 -0.00606218 -0.0735" rpy="1.5708 8.1119e-15 -0.523599"/>
     <parent link="shaft"/>
     <child link="lin_2_br"/>
     <axis xyz="0 0 -1"/>
-    <limit effort="10" velocity="10" lower="-6.281592653589793" upper="6.281592653589793"/>
+    <limit effort="10" velocity="10" lower="-3.141592653589793" upper="3.141592653589793"/>
   </joint>
   <!-- Joint from motor to shaft -->
   <joint name="joint_br_1" type="revolute">
-    <origin xyz="-0.055 0.0342754 0.061" rpy="3.14159 4.55869e-16 -1.5708"/>
+    <origin xyz="-0.055 0.0342754 0.061" rpy="-3.14159 -2.04333e-29 -1.5708"/>
     <parent link="motor"/>
     <child link="shaft"/>
     <axis xyz="0 0 -1"/>
-    <limit effort="10" velocity="10" lower="-6.281592653589793" upper="6.281592653589793"/>
+    <limit effort="10" velocity="10" lower="-3.141592653589793" upper="3.141592653589793"/>
   </joint>
   <!-- Link shaft_2 -->
   <link name="shaft_2">
     <inertial>
-      <origin xyz="0.000552419 0.00826087 -0.0535667" rpy="0 0 0"/>
+      <origin xyz="-0.00365203 0.00743033 -0.0535667" rpy="0 0 0"/>
       <mass value="0.500834"/>
-      <inertia ixx="0.000632059" ixy="-3.82058e-06" ixz="1.6979e-06" iyy="0.000740174" iyz="3.83796e-05" izz="0.000280763"/>
+      <inertia ixx="0.000662397" ixy="-4.87254e-05" ixz="-1.77194e-05" iyy="0.000709837" iyz="3.40867e-05" izz="0.000280763"/>
     </inertial>
     <!-- Part shaft_4 -->
@@ -401,5 +402,5 @@
     <!-- Part motor_5 -->
     <visual>
-      <origin xyz="0 0.017 -0.0735" rpy="1.5708 1.58313e-16 -1.5708"/>
+      <origin xyz="-0.0085 0.0147224 -0.0735" rpy="1.5708 8.92383e-17 -1.0472"/>
       <geometry>
         <mesh filename="file://$(find quadro)/description/leg_assets/motor.stl"/>
@@ -410,5 +411,5 @@
     </visual>
     <collision>
-      <origin xyz="0 0.017 -0.0735" rpy="1.5708 1.58313e-16 -1.5708"/>
+      <origin xyz="-0.0085 0.0147224 -0.0735" rpy="1.5708 8.92383e-17 -1.0472"/>
       <geometry>
         <mesh filename="file://$(find quadro)/description/leg_assets/motor.stl"/>
@@ -417,5 +418,5 @@
     <!-- Part lin_1_support_bl -->
     <visual>
-      <origin xyz="6.93889e-18 0.097 -0.0735" rpy="3.14159 -1.5708 0"/>
+      <origin xyz="-0.0485 0.0840045 -0.0735" rpy="-2.61799 -1.5708 0"/>
       <geometry>
         <mesh filename="file://$(find quadro)/description/leg_assets/lin_1_support_bl.stl"/>
@@ -426,5 +427,5 @@
     </visual>
     <collision>
-      <origin xyz="6.93889e-18 0.097 -0.0735" rpy="3.14159 -1.5708 0"/>
+      <origin xyz="-0.0485 0.0840045 -0.0735" rpy="-2.61799 -1.5708 0"/>
       <geometry>
         <mesh filename="file://$(find quadro)/description/leg_assets/lin_1_support_bl.stl"/>
@@ -441,5 +442,5 @@
     <!-- Part lin_3_top_l -->
     <visual>
-      <origin xyz="8.32667e-16 4.16334e-16 0.087" rpy="-1.5708 7.63748e-16 -1.22173"/>
+      <origin xyz="6.52256e-16 1.11022e-16 0.087" rpy="-1.5708 7.28298e-16 -1.22173"/>
       <geometry>
         <mesh filename="file://$(find quadro)/description/leg_assets/lin_3_top_l.stl"/>
@@ -450,5 +451,5 @@
     </visual>
     <collision>
-      <origin xyz="8.32667e-16 4.16334e-16 0.087" rpy="-1.5708 7.63748e-16 -1.22173"/>
+      <origin xyz="6.52256e-16 1.11022e-16 0.087" rpy="-1.5708 7.28298e-16 -1.22173"/>
       <geometry>
         <mesh filename="file://$(find quadro)/description/leg_assets/lin_3_top_l.stl"/>
@@ -457,5 +458,5 @@
     <!-- Part lin_2_bl -->
     <visual>
-      <origin xyz="6.93889e-18 2.77556e-17 -0.0195" rpy="1.5708 3.2918e-17 1.13446"/>
+      <origin xyz="-6.93889e-18 -5.55112e-17 -0.0195" rpy="1.5708 4.12056e-17 1.13446"/>
       <geometry>
         <mesh filename="file://$(find quadro)/description/leg_assets/lin_2_bl.stl"/>
@@ -466,5 +467,5 @@
     </visual>
     <collision>
-      <origin xyz="6.93889e-18 2.77556e-17 -0.0195" rpy="1.5708 3.2918e-17 1.13446"/>
+      <origin xyz="-6.93889e-18 -5.55112e-17 -0.0195" rpy="1.5708 4.12056e-17 1.13446"/>
       <geometry>
         <mesh filename="file://$(find quadro)/description/leg_assets/lin_2_bl.stl"/>
@@ -473,5 +474,5 @@
     <!-- Part lin_3_bot_l -->
     <visual>
-      <origin xyz="7.07767e-16 1.11022e-16 0.087" rpy="-1.5708 -4.29742e-16 -1.22173"/>
+      <origin xyz="6.80012e-16 5.55112e-17 0.087" rpy="-1.5708 -4.65192e-16 -1.22173"/>
       <geometry>
         <mesh filename="file://$(find quadro)/description/leg_assets/lin_3_bot_l.stl"/>
@@ -482,5 +483,5 @@
     </visual>
     <collision>
-      <origin xyz="7.07767e-16 1.11022e-16 0.087" rpy="-1.5708 -4.29742e-16 -1.22173"/>
+      <origin xyz="6.80012e-16 5.55112e-17 0.087" rpy="-1.5708 -4.65192e-16 -1.22173"/>
       <geometry>
         <mesh filename="file://$(find quadro)/description/leg_assets/lin_3_bot_l.stl"/>
@@ -489,5 +490,5 @@
     <!-- Part shaft_5 -->
     <visual>
-      <origin xyz="-6.93889e-18 0 0.01" rpy="1.5708 1.5708 0"/>
+      <origin xyz="0 0 0.01" rpy="1.5708 1.5708 0"/>
       <geometry>
         <mesh filename="file://$(find quadro)/description/leg_assets/shaft.stl"/>
@@ -498,5 +499,5 @@
     </visual>
     <collision>
-      <origin xyz="-6.93889e-18 0 0.01" rpy="1.5708 1.5708 0"/>
+      <origin xyz="0 0 0.01" rpy="1.5708 1.5708 0"/>
       <geometry>
         <mesh filename="file://$(find quadro)/description/leg_assets/shaft.stl"/>
@@ -505,5 +506,5 @@
     <!-- Part motor_6 -->
     <visual>
-      <origin xyz="9.08995e-16 8.32667e-17 -0.0385" rpy="-2.70526 1.5708 0"/>
+      <origin xyz="8.95117e-16 2.77556e-17 -0.0385" rpy="-2.70526 1.5708 0"/>
       <geometry>
         <mesh filename="file://$(find quadro)/description/leg_assets/motor.stl"/>
@@ -514,5 +515,5 @@
     </visual>
     <collision>
-      <origin xyz="9.08995e-16 8.32667e-17 -0.0385" rpy="-2.70526 1.5708 0"/>
+      <origin xyz="8.95117e-16 2.77556e-17 -0.0385" rpy="-2.70526 1.5708 0"/>
       <geometry>
         <mesh filename="file://$(find quadro)/description/leg_assets/motor.stl"/>
@@ -529,5 +530,5 @@
     <!-- Part shaft_6 -->
     <visual>
-      <origin xyz="1.04083e-17 0 0.01" rpy="1.5708 1.5708 0"/>
+      <origin xyz="8.67362e-18 2.77556e-17 0.01" rpy="1.5708 1.5708 0"/>
       <geometry>
         <mesh filename="file://$(find quadro)/description/leg_assets/shaft.stl"/>
@@ -538,5 +539,5 @@
     </visual>
     <collision>
-      <origin xyz="1.04083e-17 0 0.01" rpy="1.5708 1.5708 0"/>
+      <origin xyz="8.67362e-18 2.77556e-17 0.01" rpy="1.5708 1.5708 0"/>
       <geometry>
         <mesh filename="file://$(find quadro)/description/leg_assets/shaft.stl"/>
@@ -545,5 +546,5 @@
     <!-- Part bearing_4 -->
     <visual>
-      <origin xyz="0.0353553 0.0353553 -0.0255" rpy="3.14159 1.92161e-16 -0.785398"/>
+      <origin xyz="0.0353553 0.0353553 -0.0255" rpy="3.14159 2.00877e-16 -0.785398"/>
       <geometry>
         <mesh filename="file://$(find quadro)/description/leg_assets/bearing.stl"/>
@@ -554,5 +555,5 @@
     </visual>
     <collision>
-      <origin xyz="0.0353553 0.0353553 -0.0255" rpy="3.14159 1.92161e-16 -0.785398"/>
+      <origin xyz="0.0353553 0.0353553 -0.0255" rpy="3.14159 2.00877e-16 -0.785398"/>
       <geometry>
         <mesh filename="file://$(find quadro)/description/leg_assets/bearing.stl"/>
@@ -561,5 +562,5 @@
     <!-- Part lin_top_l -->
     <visual>
-      <origin xyz="-2.42861e-17 5.55112e-17 0.1545" rpy="-1.5708 1.3665e-16 -0.785398"/>
+      <origin xyz="-5.20417e-18 5.55112e-17 0.1545" rpy="-1.5708 1.45366e-16 -0.785398"/>
       <geometry>
         <mesh filename="file://$(find quadro)/description/leg_assets/lin_top_l.stl"/>
@@ -570,5 +571,5 @@
     </visual>
     <collision>
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