Commit message: changed model for longer legs, basic crawl now basically works, still unstable

File: description/robot_short_legs.xacro (robot description, xacro)
@@ -11,14 +11,14 @@
 </xacro:unless>
   <!-- Link motor -->
-  <!-- <link name="world"/>
+  <link name="world"/>
   <joint name="fixed" type="fixed">
     <parent link="world"/>
     <child link="back_plate"/>
-  </joint> -->
+  </joint>
   <link name="back_plate">
     <inertial>
       <origin xyz="-0.139034 0.00943483 -0.0243213" rpy="0 0 0"/>
       <mass value="2.38325"/>
-      <inertia ixx="0.0204343" ixy="-3.21203e-05" ixz="6.9264e-20" iyy="0.00715196" iyz="-4.17004e-19" izz="0.0254162"/>
+      <inertia ixx="0.0204343" ixy="-3.21203e-05" ixz="7.46306e-20" iyy="0.00715196" iyz="-4.17004e-19" izz="0.0254162"/>
     </inertial>
     <!-- Part back_stop -->
@@ -437,13 +437,12 @@
     <child link="shaft_3"/>
     <axis xyz="0 0 -1"/>
-    <limit effort="40" velocity="12" lower="-3.141592653589793" upper="3.141592653589793"/>
-    <joint_properties friction="0.5"/>
+    <limit effort="20" velocity="10" lower="-3.141592653589793" upper="3.141592653589793"/>
   </joint>
   <!-- Link lin_4_r -->
   <link name="lin_4_r">
     <inertial>
-      <origin xyz="-0.000262324 0.0491557 -0.0035" rpy="0 0 0"/>
-      <mass value="0.0701023"/>
-      <inertia ixx="0.000371839" ixy="-2.10379e-06" ixz="-2.70636e-13" iyy="6.27155e-06" iyz="2.29312e-12" izz="0.000376266"/>
+      <origin xyz="-0.000162389 0.0733841 -0.0035" rpy="0 0 0"/>
+      <mass value="0.0813924"/>
+      <inertia ixx="0.000647132" ixy="-2.74301e-06" ixz="-2.68991e-13" iyy="7.272e-06" iyz="2.78217e-12" izz="0.000652467"/>
     </inertial>
     <!-- Part lin_4_r -->
@@ -518,6 +517,5 @@
     <child link="lin_4_r"/>
     <axis xyz="0 0 -1"/>
-    <limit effort="40" velocity="12" lower="-3.141592653589793" upper="3.141592653589793"/>
-    <joint_properties friction="0.5"/>
+    <limit effort="20" velocity="10" lower="-3.141592653589793" upper="3.141592653589793"/>
     <mimic joint="br_m3_s3" multiplier="1.0"/>
   </joint>
@@ -528,6 +526,5 @@
     <child link="shaft_2"/>
     <axis xyz="0 0 -1"/>
-    <limit effort="40" velocity="12" lower="-3.141592653589793" upper="3.141592653589793"/>
-    <joint_properties friction="0.5"/>
+    <limit effort="20" velocity="10" lower="-3.141592653589793" upper="3.141592653589793"/>
   </joint>
   <!-- Joint from back_plate to shaft -->
@@ -537,6 +534,5 @@
     <child link="shaft"/>
     <axis xyz="0 0 -1"/>
-    <limit effort="40" velocity="12" lower="-3.141592653589793" upper="3.141592653589793"/>
-    <joint_properties friction="0.5"/>
+    <limit effort="20" velocity="10" lower="-3.141592653589793" upper="3.141592653589793"/>
   </joint>
   <!-- Link shaft_4 -->
@@ -746,13 +742,12 @@
     <child link="shaft_6"/>
     <axis xyz="0 0 1"/>
-    <limit effort="40" velocity="12" lower="-3.141592653589793" upper="3.141592653589793"/>
-    <joint_properties friction="0.5"/>
+    <limit effort="20" velocity="10" lower="-3.141592653589793" upper="3.141592653589793"/>
   </joint>
   <!-- Link lin_4_l -->
   <link name="lin_4_l">
     <inertial>
-      <origin xyz="-0.000262328 -0.0491558 -0.0035" rpy="0 0 0"/>
-      <mass value="0.0701023"/>
-      <inertia ixx="0.000371839" ixy="2.10381e-06" ixz="2.70636e-13" iyy="6.27154e-06" iyz="2.29312e-12" izz="0.000376266"/>
+      <origin xyz="-0.000162393 -0.0733841 -0.0035" rpy="0 0 0"/>
+      <mass value="0.0813924"/>
+      <inertia ixx="0.000647132" ixy="2.74304e-06" ixz="2.68991e-13" iyy="7.272e-06" iyz="2.78217e-12" izz="0.000652466"/>
     </inertial>
     <!-- Part bearing_5 -->
@@ -827,6 +822,5 @@
     <child link="lin_4_l"/>
     <axis xyz="0 0 1"/>
-    <limit effort="40" velocity="12" lower="-3.141592653589793" upper="3.141592653589793"/>
-    <joint_properties friction="0.5"/>
+    <limit effort="20" velocity="10" lower="-3.141592653589793" upper="3.141592653589793"/>
     <mimic joint="bl_m3_s3" multiplier="1.0"/>
   </joint>
@@ -837,6 +831,5 @@
     <child link="shaft_5"/>
     <axis xyz="0 0 1"/>
-    <limit effort="40" velocity="12" lower="-3.141592653589793" upper="3.141592653589793"/>
-    <joint_properties friction="0.5"/>
+    <limit effort="20" velocity="10" lower="-3.141592653589793" upper="3.141592653589793"/>
   </joint>
   <!-- Joint from back_plate to shaft_4 -->
@@ -846,6 +839,5 @@
     <child link="shaft_4"/>
     <axis xyz="0 0 -1"/>
-    <limit effort="40" velocity="12" lower="-3.141592653589793" upper="3.141592653589793"/>
-    <joint_properties friction="0.5"/>
+    <limit effort="20" velocity="10" lower="-3.141592653589793" upper="3.141592653589793"/>
   </joint>
   <!-- Link shaft_7 -->
@@ -1055,13 +1047,12 @@
     <child link="shaft_9"/>
     <axis xyz="0 0 -1"/>
-    <limit effort="40" velocity="12" lower="-3.141592653589793" upper="3.141592653589793"/>
-    <joint_properties friction="0.5"/>
+    <limit effort="20" velocity="10" lower="-3.141592653589793" upper="3.141592653589793"/>
   </joint>
   <!-- Link lin_4_r_2 -->
   <link name="lin_4_r_2">
     <inertial>
-      <origin xyz="-0.000262324 0.0491557 -0.0035" rpy="0 0 0"/>
-      <mass value="0.0701023"/>
-      <inertia ixx="0.000371839" ixy="-2.10379e-06" ixz="-2.70636e-13" iyy="6.27155e-06" iyz="2.29312e-12" izz="0.000376266"/>
+      <origin xyz="-0.000162389 0.0733841 -0.0035" rpy="0 0 0"/>
+      <mass value="0.0813924"/>
+      <inertia ixx="0.000647132" ixy="-2.74301e-06" ixz="-2.68991e-13" iyy="7.272e-06" iyz="2.78217e-12" izz="0.000652467"/>
     </inertial>
     <!-- Part bearing_8 -->
@@ -1136,6 +1127,5 @@
     <child link="lin_4_r_2"/>
     <axis xyz="0 0 -1"/>
-    <limit effort="40" velocity="12" lower="-3.141592653589793" upper="3.141592653589793"/>
-    <joint_properties friction="0.5"/>
+    <limit effort="20" velocity="10" lower="-3.141592653589793" upper="3.141592653589793"/>
     <mimic joint="fr_m3_s3" multiplier="1.0"/>
   </joint>
@@ -1146,6 +1136,5 @@
     <child link="shaft_8"/>
     <axis xyz="0 0 -1"/>
-    <limit effort="40" velocity="12" lower="-3.141592653589793" upper="3.141592653589793"/>
-    <joint_properties friction="0.5"/>
+    <limit effort="20" velocity="10" lower="-3.141592653589793" upper="3.141592653589793"/>
   </joint>
   <!-- Joint from back_plate to shaft_7 -->
@@ -1155,6 +1144,5 @@
     <child link="shaft_7"/>
     <axis xyz="0 0 1"/>
-    <limit effort="40" velocity="12" lower="-3.141592653589793" upper="3.141592653589793"/>
-    <joint_properties friction="0.5"/>
+    <limit effort="20" velocity="10" lower="-3.141592653589793" upper="3.141592653589793"/>
   </joint>
   <!-- Link motor -->
@@ -1364,13 +1352,12 @@
     <child link="shaft_10"/>
     <axis xyz="0 0 1"/>
-    <limit effort="40" velocity="12" lower="-3.141592653589793" upper="3.141592653589793"/>
-    <joint_properties friction="0.5"/>
+    <limit effort="20" velocity="10" lower="-3.141592653589793" upper="3.141592653589793"/>
   </joint>
   <!-- Link lin_4_l_2 -->
   <link name="lin_4_l_2">
     <inertial>
-      <origin xyz="-0.000262328 -0.0491558 -0.0035" rpy="0 0 0"/>
-      <mass value="0.0701023"/>
-      <inertia ixx="0.000371839" ixy="2.10381e-06" ixz="2.70636e-13" iyy="6.27154e-06" iyz="2.29312e-12" izz="0.000376266"/>
+      <origin xyz="-0.000162393 -0.0733841 -0.0035" rpy="0 0 0"/>
+      <mass value="0.0813924"/>
+      <inertia ixx="0.000647132" ixy="2.74304e-06" ixz="2.68991e-13" iyy="7.272e-06" iyz="2.78217e-12" izz="0.000652466"/>
     </inertial>
     <!-- Part feet_4 -->
@@ -1445,6 +1432,5 @@
     <child link="lin_4_l_2"/>
     <axis xyz="0 0 1"/>
-    <limit effort="40" velocity="12" lower="-3.141592653589793" upper="3.141592653589793"/>
-    <joint_properties friction="0.5"/>
+    <limit effort="20" velocity="10" lower="-3.141592653589793" upper="3.141592653589793"/>
     <mimic joint="fl_m3_s3" multiplier="1.0"/>
   </joint>
@@ -1455,6 +1441,5 @@
     <child link="motor_2"/>
     <axis xyz="0 0 1"/>
-    <limit effort="40" velocity="12" lower="-3.141592653589793" upper="3.141592653589793"/>
-    <joint_properties friction="0.5"/>
+    <limit effort="20" velocity="10" lower="-3.141592653589793" upper="3.141592653589793"/>
   </joint>
   <!-- Joint from back_plate to motor -->
@@ -1464,6 +1449,5 @@
     <child link="motor"/>
     <axis xyz="0 0 1"/>
-    <limit effort="40" velocity="12" lower="-3.141592653589793" upper="3.141592653589793"/>
-    <joint_properties friction="0.5"/>
+    <limit effort="20" velocity="10" lower="-3.141592653589793" upper="3.141592653589793"/>
   </joint>
 </robot>
