Commit message: added rotation when walking

File: description/robot.xacro (robot description, xacro)
@@ -14,5 +14,5 @@
   <joint name="fixed" type="fixed">
     <parent link="world"/>
-    <child link="motor"/>
+    <child link="back_plate"/>
   </joint> -->
   <link name="back_plate">
@@ -437,5 +437,5 @@
     <child link="shaft_3"/>
     <axis xyz="0 0 -1"/>
-    <limit effort="10" velocity="12" lower="-3.141592653589793" upper="3.141592653589793"/>
+    <limit effort="20" velocity="12" lower="-3.141592653589793" upper="3.141592653589793"/>
     <joint_properties friction="0.5"/>
   </joint>
@@ -518,5 +518,5 @@
     <child link="lin_4_r"/>
     <axis xyz="0 0 -1"/>
-    <limit effort="10" velocity="12" lower="-3.141592653589793" upper="3.141592653589793"/>
+    <limit effort="20" velocity="12" lower="-3.141592653589793" upper="3.141592653589793"/>
     <joint_properties friction="0.5"/>
     <mimic joint="br_m3_s3" multiplier="1.0"/>
@@ -528,5 +528,5 @@
     <child link="shaft_2"/>
     <axis xyz="0 0 -1"/>
-    <limit effort="10" velocity="12" lower="-3.141592653589793" upper="3.141592653589793"/>
+    <limit effort="20" velocity="12" lower="-3.141592653589793" upper="3.141592653589793"/>
     <joint_properties friction="0.5"/>
   </joint>
@@ -537,5 +537,5 @@
     <child link="shaft"/>
     <axis xyz="0 0 -1"/>
-    <limit effort="10" velocity="12" lower="-3.141592653589793" upper="3.141592653589793"/>
+    <limit effort="20" velocity="12" lower="-3.141592653589793" upper="3.141592653589793"/>
     <joint_properties friction="0.5"/>
   </joint>
@@ -746,5 +746,5 @@
     <child link="shaft_6"/>
     <axis xyz="0 0 1"/>
-    <limit effort="10" velocity="12" lower="-3.141592653589793" upper="3.141592653589793"/>
+    <limit effort="20" velocity="12" lower="-3.141592653589793" upper="3.141592653589793"/>
     <joint_properties friction="0.5"/>
   </joint>
@@ -827,5 +827,5 @@
     <child link="lin_4_l"/>
     <axis xyz="0 0 1"/>
-    <limit effort="10" velocity="12" lower="-3.141592653589793" upper="3.141592653589793"/>
+    <limit effort="20" velocity="12" lower="-3.141592653589793" upper="3.141592653589793"/>
     <joint_properties friction="0.5"/>
     <mimic joint="bl_m3_s3" multiplier="1.0"/>
@@ -837,5 +837,5 @@
     <child link="shaft_5"/>
     <axis xyz="0 0 1"/>
-    <limit effort="10" velocity="12" lower="-3.141592653589793" upper="3.141592653589793"/>
+    <limit effort="20" velocity="12" lower="-3.141592653589793" upper="3.141592653589793"/>
     <joint_properties friction="0.5"/>
   </joint>
@@ -846,5 +846,5 @@
     <child link="shaft_4"/>
     <axis xyz="0 0 -1"/>
-    <limit effort="10" velocity="12" lower="-3.141592653589793" upper="3.141592653589793"/>
+    <limit effort="20" velocity="12" lower="-3.141592653589793" upper="3.141592653589793"/>
     <joint_properties friction="0.5"/>
   </joint>
@@ -1055,5 +1055,5 @@
     <child link="shaft_9"/>
     <axis xyz="0 0 -1"/>
-    <limit effort="10" velocity="12" lower="-3.141592653589793" upper="3.141592653589793"/>
+    <limit effort="20" velocity="12" lower="-3.141592653589793" upper="3.141592653589793"/>
     <joint_properties friction="0.5"/>
   </joint>
@@ -1136,5 +1136,5 @@
     <child link="lin_4_r_2"/>
     <axis xyz="0 0 -1"/>
-    <limit effort="10" velocity="12" lower="-3.141592653589793" upper="3.141592653589793"/>
+    <limit effort="20" velocity="12" lower="-3.141592653589793" upper="3.141592653589793"/>
     <joint_properties friction="0.5"/>
     <mimic joint="fr_m3_s3" multiplier="1.0"/>
@@ -1146,5 +1146,5 @@
     <child link="shaft_8"/>
     <axis xyz="0 0 -1"/>
-    <limit effort="10" velocity="12" lower="-3.141592653589793" upper="3.141592653589793"/>
+    <limit effort="20" velocity="12" lower="-3.141592653589793" upper="3.141592653589793"/>
     <joint_properties friction="0.5"/>
   </joint>
@@ -1155,5 +1155,5 @@
     <child link="shaft_7"/>
     <axis xyz="0 0 1"/>
-    <limit effort="10" velocity="12" lower="-3.141592653589793" upper="3.141592653589793"/>
+    <limit effort="20" velocity="12" lower="-3.141592653589793" upper="3.141592653589793"/>
     <joint_properties friction="0.5"/>
   </joint>
@@ -1364,5 +1364,5 @@
     <child link="shaft_10"/>
     <axis xyz="0 0 1"/>
-    <limit effort="10" velocity="12" lower="-3.141592653589793" upper="3.141592653589793"/>
+    <limit effort="20" velocity="12" lower="-3.141592653589793" upper="3.141592653589793"/>
     <joint_properties friction="0.5"/>
   </joint>
@@ -1445,5 +1445,5 @@
     <child link="lin_4_l_2"/>
     <axis xyz="0 0 1"/>
-    <limit effort="10" velocity="12" lower="-3.141592653589793" upper="3.141592653589793"/>
+    <limit effort="20" velocity="12" lower="-3.141592653589793" upper="3.141592653589793"/>
     <joint_properties friction="0.5"/>
     <mimic joint="fl_m3_s3" multiplier="1.0"/>
@@ -1455,5 +1455,5 @@
     <child link="motor_2"/>
     <axis xyz="0 0 1"/>
-    <limit effort="10" velocity="12" lower="-3.141592653589793" upper="3.141592653589793"/>
+    <limit effort="20" velocity="12" lower="-3.141592653589793" upper="3.141592653589793"/>
     <joint_properties friction="0.5"/>
   </joint>
@@ -1464,5 +1464,5 @@
     <child link="motor"/>
     <axis xyz="0 0 1"/>
-    <limit effort="10" velocity="12" lower="-3.141592653589793" upper="3.141592653589793"/>
+    <limit effort="20" velocity="12" lower="-3.141592653589793" upper="3.141592653589793"/>
     <joint_properties friction="0.5"/>
   </joint>
