Commit message: started integration with hardware

File: description/one_motor_control.xacro (robot description, xacro)
@@ -6,10 +6,10 @@
       <param name="can">can0</param>
     </hardware>
-    <joint name="BR1">
+    <joint name="br_m1_s1">
       <command_interface name="position">
       </command_interface>
       <state_interface name="position"/>
       <state_interface name="velocity"/>
-      <param name="node_id">0</param>
+      <param name="node_id">9</param>
     </joint>
     <!-- <transmission name="br1_trans">

File: description/quadro.xacro (robot description, xacro)
@@ -10,110 +10,1454 @@
   <xacro:include filename="$(find quadro)/description/ros2_control.xacro" />
 </xacro:unless>
-<link name="world"></link>
-<link name="base_link">
-  <inertial>
-    <origin xyz="-0.000584411215524606 0.00012078668947847333 0.020036075822933482" rpy="0 0 0"/>
-    <mass value="0.8821101167454488"/>
-    <inertia ixx="0.000352" iyy="0.000363" izz="0.000583" ixy="3e-06" iyz="0.0" ixz="-0.0"/>
-  </inertial>
-  <visual>
-    <origin xyz="0 0 0" rpy="0 0 0"/>
-    <geometry>
-      <mesh filename="file://$(find quadro)/description/meshes/base_link.stl" scale="0.001 0.001 0.001"/>
-    </geometry>
-    <material name="silver"/>
-  </visual>
-  <collision>
-    <origin xyz="0 0 0" rpy="0 0 0"/>
-    <geometry>
-      <mesh filename="file://$(find quadro)/description/meshes/base_link.stl" scale="0.001 0.001 0.001"/>
-    </geometry>
-  </collision>
-</link>
-<link name="link_1_1">
-  <inertial>
-    <origin xyz="-0.012749021534557922 0.0001313434135850603 0.04451702298542016" rpy="0 0 0"/>
-    <mass value="1.621189326543191"/>
-    <inertia ixx="0.001785" iyy="0.001338" izz="0.000977" ixy="2e-06" iyz="6e-06" ixz="-1.2e-05"/>
-  </inertial>
-  <visual>
-    <origin xyz="0.000251 -7e-06 -0.0365" rpy="0 0 0"/>
-    <geometry>
-      <mesh filename="file://$(find quadro)/description/meshes/link_1_1.stl" scale="0.001 0.001 0.001"/>
-    </geometry>
-    <material name="silver"/>
-  </visual>
-  <collision>
-    <origin xyz="0.000251 -7e-06 -0.0365" rpy="0 0 0"/>
-    <geometry>
-      <mesh filename="file://$(find quadro)/description/meshes/link_1_1.stl" scale="0.001 0.001 0.001"/>
-    </geometry>
-  </collision>
-</link>
-<link name="link_2_1">
-  <inertial>
-    <origin xyz="0.025429277256362695 -0.008464137973570403 0.008149150240915351" rpy="0 0 0"/>
-    <mass value="1.5970767317820915"/>
-    <inertia ixx="0.003865" iyy="0.002207" izz="0.002316" ixy="0.00029" iyz="0.001344" ixz="-0.00026"/>
-  </inertial>
-  <visual>
-    <origin xyz="-0.010269 0.000144 -0.090593" rpy="0 0 0"/>
-    <geometry>
-      <mesh filename="file://$(find quadro)/description/meshes/link_2_1.stl" scale="0.001 0.001 0.001"/>
-    </geometry>
-    <material name="silver"/>
-  </visual>
-  <collision>
-    <origin xyz="-0.010269 0.000144 -0.090593" rpy="0 0 0"/>
-    <geometry>
-      <mesh filename="file://$(find quadro)/description/meshes/link_2_1.stl" scale="0.001 0.001 0.001"/>
-    </geometry>
-  </collision>
-</link>
-<link name="link_3_1">
-  <inertial>
-    <origin xyz="0.003501872886119403 -0.04049316234641598 -0.0005238984066143759" rpy="0 0 0"/>
-    <mass value="0.2609392030209961"/>
-    <inertia ixx="0.000861" iyy="2.8e-05" izz="0.000835" ixy="-0.0" iyz="1.3e-05" ixz="-0.0"/>
-  </inertial>
-  <visual>
-    <origin xyz="-0.056769 0.141957 -0.232219" rpy="0 0 0"/>
-    <geometry>
-      <mesh filename="file://$(find quadro)/description/meshes/link_3_1.stl" scale="0.001 0.001 0.001"/>
-    </geometry>
-    <material name="silver"/>
-  </visual>
-  <collision>
-    <origin xyz="-0.056769 0.141957 -0.232219" rpy="0 0 0"/>
-    <geometry>
-      <mesh filename="file://$(find quadro)/description/meshes/link_3_1.stl" scale="0.001 0.001 0.001"/>
-    </geometry>
-  </collision>
-</link>
-<joint name="base_joint" type="fixed">
-    <origin xyz="0.0 0.0 -0.07" rpy="0 0 0"/>
-    <parent link="world"/>
-    <child link="base_link"/>
-</joint>
-<joint name="BR1" type="continuous">
-  <origin xyz="-0.000251 7e-06 0.0365" rpy="0 0 0"/>
-  <parent link="base_link"/>
-  <child link="link_1_1"/>
-  <axis xyz="0.0 0.0 -1.0"/>
-  <limit effort="12" velocity="2" lower="-1.57" upper="1.57"/>
-</joint>
-<joint name="BR2" type="continuous">
-  <origin xyz="0.01052 -0.000151 0.054093" rpy="0 0 0"/>
-  <parent link="link_1_1"/>
-  <child link="link_2_1"/>
-  <axis xyz="-1.0 0.0 0.0"/>
-  <limit effort="120" velocity="4" lower="0.0" upper="1.20"/>
-</joint>
-<joint name="BR3" type="continuous">
-  <origin xyz="0.0465 -0.141813 0.141626" rpy="0 0 0"/>
-  <parent link="link_2_1"/>
-  <child link="link_3_1"/>
-  <axis xyz="-1.0 0.0 0.0"/>
-  <limit effort="120" velocity="4" lower="0.0" upper="1.20"/>
-</joint>
+  <link name="back_plate">
+    <inertial>
+      <origin xyz="-0.139034 0.00943483 -0.0243213" rpy="0 0 0"/>
+      <mass value="2.38325"/>
+      <inertia ixx="0.0204343" ixy="-3.21203e-05" ixz="6.24877e-20" iyy="0.00715196" iyz="-3.89899e-19" izz="0.0254162"/>
+    </inertial>
+    <!-- Part back_stop -->
+    <visual>
+      <origin xyz="-0.139034 -0.0331652 -0.058441" rpy="0 -0 0"/>
+      <geometry>
+        <mesh filename="file://$(find quadro)/description/assets/back_stop.stl"/>
+      </geometry>
+      <material name="back_stop_material">
+        <color rgba="1 0.756863 0.054902 1"/>
+      </material>
+    </visual>
+    <collision>
+      <origin xyz="-0.139034 -0.0331652 -0.058441" rpy="0 -0 0"/>
+      <geometry>
+        <mesh filename="file://$(find quadro)/description/assets/back_stop.stl"/>
+      </geometry>
+    </collision>
+    <!-- Part side_pipe -->
+    <visual>
+      <origin xyz="-0.0083688 0.0999348 -0.058441" rpy="0 -0 0"/>
+      <geometry>
+        <mesh filename="file://$(find quadro)/description/assets/side_pipe.stl"/>
+      </geometry>
+      <material name="side_pipe_material">
+        <color rgba="0 0 0 1"/>
+      </material>
+    </visual>
+    <collision>
+      <origin xyz="-0.0083688 0.0999348 -0.058441" rpy="0 -0 0"/>
+      <geometry>
+        <mesh filename="file://$(find quadro)/description/assets/side_pipe.stl"/>
+      </geometry>
+    </collision>
+    <!-- Part back_plate -->
+    <visual>
+      <origin xyz="-0.139034 0.0999348 -0.058441" rpy="0 -0 0"/>
+      <geometry>
+        <mesh filename="file://$(find quadro)/description/assets/back_plate.stl"/>
+      </geometry>
+      <material name="back_plate_material">
+        <color rgba="1 0.756863 0.054902 1"/>
+      </material>
+    </visual>
+    <collision>
+      <origin xyz="-0.139034 0.0999348 -0.058441" rpy="0 -0 0"/>
+      <geometry>
+        <mesh filename="file://$(find quadro)/description/assets/back_plate.stl"/>
+      </geometry>
+    </collision>
+    <!-- Part battery -->
+    <visual>
+      <origin xyz="-0.0725337 -0.0125652 -0.028441" rpy="0 -6.12323e-17 1.5708"/>
+      <geometry>
+        <mesh filename="file://$(find quadro)/description/assets/battery.stl"/>
+      </geometry>
+      <material name="battery_material">
+        <color rgba="0.768627 0.886275 0.952941 1"/>
+      </material>
+    </visual>
+    <collision>
+      <origin xyz="-0.0725337 -0.0125652 -0.028441" rpy="0 -6.12323e-17 1.5708"/>
+      <geometry>
+        <mesh filename="file://$(find quadro)/description/assets/battery.stl"/>
+      </geometry>
+    </collision>
+    <!-- Part motor -->
+    <visual>
+      <origin xyz="-0.194034 -0.0920652 -0.023441" rpy="3.14159 5.95406e-36 -1.5708"/>
+      <geometry>
+        <mesh filename="file://$(find quadro)/description/assets/motor.stl"/>
+      </geometry>
+      <material name="motor_material">
+        <color rgba="0.498039 0.498039 0.498039 1"/>
+      </material>
+    </visual>
+    <collision>
+      <origin xyz="-0.194034 -0.0920652 -0.023441" rpy="3.14159 5.95406e-36 -1.5708"/>
+      <geometry>
+        <mesh filename="file://$(find quadro)/description/assets/motor.stl"/>
+      </geometry>
+    </collision>
+    <!-- Part motor_2 -->
+    <visual>
+      <origin xyz="-0.194034 0.110935 -0.023441" rpy="3.14159 5.95406e-36 1.5708"/>
+      <geometry>
+        <mesh filename="file://$(find quadro)/description/assets/motor.stl"/>
+      </geometry>
+      <material name="motor_2_material">
+        <color rgba="0.498039 0.498039 0.498039 1"/>
+      </material>
+    </visual>
+    <collision>
+      <origin xyz="-0.194034 0.110935 -0.023441" rpy="3.14159 5.95406e-36 1.5708"/>
+      <geometry>
+        <mesh filename="file://$(find quadro)/description/assets/motor.stl"/>
+      </geometry>
+    </collision>
+    <!-- Part motor_3 -->
+    <visual>
+      <origin xyz="-0.0840337 -0.0920652 -0.023441" rpy="3.14159 5.95406e-36 -1.5708"/>
+      <geometry>
+        <mesh filename="file://$(find quadro)/description/assets/motor.stl"/>
+      </geometry>
+      <material name="motor_3_material">
+        <color rgba="0.498039 0.498039 0.498039 1"/>
+      </material>
+    </visual>
+    <collision>
+      <origin xyz="-0.0840337 -0.0920652 -0.023441" rpy="3.14159 5.95406e-36 -1.5708"/>
+      <geometry>
+        <mesh filename="file://$(find quadro)/description/assets/motor.stl"/>
+      </geometry>
+    </collision>
+    <!-- Part side_pipe_2 -->
+    <visual>
+      <origin xyz="-0.139034 -0.0810652 0.0614484" rpy="3.14159 -0 0"/>
+      <geometry>
+        <mesh filename="file://$(find quadro)/description/assets/side_pipe.stl"/>
+      </geometry>
+      <material name="side_pipe_2_material">
+        <color rgba="0 0 0 1"/>
+      </material>
+    </visual>
+    <collision>
+      <origin xyz="-0.139034 -0.0810652 0.0614484" rpy="3.14159 -0 0"/>
+      <geometry>
+        <mesh filename="file://$(find quadro)/description/assets/side_pipe.stl"/>
+      </geometry>
+    </collision>
+    <!-- Part motor_4 -->
+    <visual>
+      <origin xyz="-0.0840337 0.110935 -0.023441" rpy="3.14159 5.95406e-36 1.5708"/>
+      <geometry>
+        <mesh filename="file://$(find quadro)/description/assets/motor.stl"/>
+      </geometry>
+      <material name="motor_4_material">
+        <color rgba="0.498039 0.498039 0.498039 1"/>
+      </material>
+    </visual>
+    <collision>
+      <origin xyz="-0.0840337 0.110935 -0.023441" rpy="3.14159 5.95406e-36 1.5708"/>
+      <geometry>
+        <mesh filename="file://$(find quadro)/description/assets/motor.stl"/>
+      </geometry>
+    </collision>
+    <!-- Part back_stop_2 -->
+    <visual>
+      <origin xyz="-0.139034 0.0520348 -0.058441" rpy="0 -0 3.14159"/>
+      <geometry>
+        <mesh filename="file://$(find quadro)/description/assets/back_stop.stl"/>
+      </geometry>
+      <material name="back_stop_2_material">
+        <color rgba="1 0.756863 0.054902 1"/>
+      </material>
+    </visual>
+    <collision>
+      <origin xyz="-0.139034 0.0520348 -0.058441" rpy="0 -0 3.14159"/>
+      <geometry>
+        <mesh filename="file://$(find quadro)/description/assets/back_stop.stl"/>
+      </geometry>
+    </collision>
+    <!-- Part back_plate_2 -->
+    <visual>
+      <origin xyz="-0.139034 -0.0810652 -0.058441" rpy="0 -0 3.14159"/>
+      <geometry>
+        <mesh filename="file://$(find quadro)/description/assets/back_plate.stl"/>
+      </geometry>
+      <material name="back_plate_2_material">
+        <color rgba="1 0.756863 0.054902 1"/>
+      </material>
+    </visual>
+    <collision>
+      <origin xyz="-0.139034 -0.0810652 -0.058441" rpy="0 -0 3.14159"/>
+      <geometry>
+        <mesh filename="file://$(find quadro)/description/assets/back_plate.stl"/>
+      </geometry>
+    </collision>
+    <!-- Part main_pipe -->
+    <visual>
+      <origin xyz="-0.139034 -0.133065 -0.058441" rpy="0 -0 0"/>
+      <geometry>
+        <mesh filename="file://$(find quadro)/description/assets/main_pipe.stl"/>
+      </geometry>
+      <material name="main_pipe_material">
+        <color rgba="0 0 0 1"/>
+      </material>
+    </visual>
+    <collision>
+      <origin xyz="-0.139034 -0.133065 -0.058441" rpy="0 -0 0"/>
+      <geometry>
+        <mesh filename="file://$(find quadro)/description/assets/main_pipe.stl"/>
+      </geometry>
+    </collision>
+    <!-- Part battery_2 -->
+    <visual>
+      <origin xyz="-0.205534 -0.0125652 -0.028441" rpy="3.14159 -6.12323e-17 1.5708"/>
+      <geometry>
+        <mesh filename="file://$(find quadro)/description/assets/battery.stl"/>
+      </geometry>
+      <material name="battery_2_material">
+        <color rgba="0.768627 0.886275 0.952941 1"/>
+      </material>
+    </visual>
+    <collision>
+      <origin xyz="-0.205534 -0.0125652 -0.028441" rpy="3.14159 -6.12323e-17 1.5708"/>
+      <geometry>
+        <mesh filename="file://$(find quadro)/description/assets/battery.stl"/>
+      </geometry>
+    </collision>
+  </link>
+  <!-- Link shaft -->
+  <link name="shaft">
+    <inertial>
+      <origin xyz="-0.00743033 0.00365203 -0.0538481" rpy="0 0 0"/>
+      <mass value="0.500834"/>
+      <inertia ixx="0.000715416" ixy="-4.87254e-05" ixz="-3.36343e-05" iyy="0.000667976" iyz="1.74582e-05" izz="0.000280763"/>
+    </inertial>
+    <!-- Part lin_1_support_br -->
+    <visual>
+      <origin xyz="-0.0242487 0.014 -0.0735" rpy="1.0472 -1.5708 0"/>
+      <geometry>
+        <mesh filename="file://$(find quadro)/description/assets/lin_1_support_br.stl"/>
+      </geometry>
+      <material name="lin_1_support_br_material">
+        <color rgba="1 0.756863 0.054902 1"/>
+      </material>
+    </visual>
+    <collision>
+      <origin xyz="-0.0242487 0.014 -0.0735" rpy="1.0472 -1.5708 0"/>
+      <geometry>
+        <mesh filename="file://$(find quadro)/description/assets/lin_1_support_br.stl"/>
+      </geometry>
+    </collision>
+    <!-- Part motor_5 -->
+    <visual>
+      <origin xyz="-0.0147224 0.0085 -0.0735" rpy="-1.5708 6.61824e-17 -0.523599"/>
+      <geometry>
+        <mesh filename="file://$(find quadro)/description/assets/motor.stl"/>
+      </geometry>
+      <material name="motor_5_material">
+        <color rgba="0.498039 0.498039 0.498039 1"/>
+      </material>
+    </visual>
+    <collision>
+      <origin xyz="-0.0147224 0.0085 -0.0735" rpy="-1.5708 6.61824e-17 -0.523599"/>
+      <geometry>
+        <mesh filename="file://$(find quadro)/description/assets/motor.stl"/>
+      </geometry>
+    </collision>
+    <!-- Part shaft -->
+    <visual>
+      <origin xyz="0 0 0.01" rpy="1.5708 1.5708 0"/>
+      <geometry>
+        <mesh filename="file://$(find quadro)/description/assets/shaft.stl"/>
+      </geometry>
+      <material name="shaft_material">
+        <color rgba="0.498039 0.498039 0.498039 1"/>
+      </material>
+    </visual>
+    <collision>
+      <origin xyz="0 0 0.01" rpy="1.5708 1.5708 0"/>
+      <geometry>
+        <mesh filename="file://$(find quadro)/description/assets/shaft.stl"/>
+      </geometry>
+    </collision>
+  </link>
+  <!-- Link shaft_2 -->
+  <link name="shaft_2">
+    <inertial>
+      <origin xyz="0.0106548 -0.00501565 -0.0435875" rpy="0 0 0"/>
+      <mass value="0.551476"/>
+      <inertia ixx="0.000599797" ixy="0.000304448" ixz="0.000186335" iyy="0.00130385" iyz="-9.91623e-05" izz="0.00132343"/>
+    </inertial>
+    <!-- Part lin_3_bot_r -->
+    <visual>
+      <origin xyz="2.77556e-17 8.04912e-16 -0.0645" rpy="1.5708 -3.60822e-16 2.79253"/>
+      <geometry>
+        <mesh filename="file://$(find quadro)/description/assets/lin_3_bot_r.stl"/>
+      </geometry>
+      <material name="lin_3_bot_r_material">
+        <color rgba="1 0.756863 0.054902 1"/>
+      </material>
+    </visual>
+    <collision>
+      <origin xyz="2.77556e-17 8.04912e-16 -0.0645" rpy="1.5708 -3.60822e-16 2.79253"/>
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
File: description/ros2_control.xacro (robot description, xacro)
@@ -1,14 +1,17 @@
 <?xml version="1.0" ?>
 <robot name="quadro" xmlns:xacro="http://www.ros.org/wiki/xacro" >
-    <ros2_control name="CybergearActuators" type="actuator">
+  <ros2_control name="motor_controller" type="system">
     <hardware>
-      <plugin>quadro/CybergearActuator</plugin>
-      <param name="can_interface">can0</param>
-      <param name="timeout_sec">3.0</param>
-      <param name="use_bus_time">false</param>
-      <param name="interval_sec">0.5</param>
-      <param name="primary_id">0</param>
+      <plugin>odrive_ros2_control_plugin/ODriveHardwareInterface</plugin>
+      <param name="can">can0</param>
     </hardware>
     <joint name="br_m1_s1">
+      <command_interface name="position">
+      </command_interface>
+      <state_interface name="position"/>
+      <state_interface name="velocity"/>
+      <param name="node_id">9</param>
+    </joint>
+    <!-- <joint name="br_m1_s1">
       <command_interface name="position">
       </command_interface>
@@ -81,5 +84,5 @@
       <state_interface name="position"/>
       <state_interface name="velocity"/>
-    </joint>
+    </joint> -->
   </ros2_control>
 </robot>
