Commit message: fixed isaac sim model

File: description/robot_full_urdf.urdf (robot description, URDF)
Before this commit: robot robot, 17 links, 16 joints
Joints:
- joint bl_m1_s1: axis 0 0 -1 -> 0 0 1
- joint br_l4_l3: axis 0 0 -1 -> 0 0 1
- joint br_m1_s1: axis 0 0 -1 -> 0 0 1
- joint br_m2_s2: axis 0 0 -1 -> 0 0 1
- joint br_m3_s3: axis 0 0 -1 -> 0 0 1
- joint fr_l4_l3: axis 0 0 -1 -> 0 0 1
- joint fr_m2_s2: axis 0 0 -1 -> 0 0 1
- joint fr_m3_s3: axis 0 0 -1 -> 0 0 1
