Commit message: isolated BR leg

File: description/ros2_control.xacro (robot description, xacro)
@@ -12,4 +12,11 @@
       <state_interface name="velocity"/>
       <param name="node_id">9</param>
+    </joint>
+    <joint name="br_m2_s2">
+      <command_interface name="position">
+      </command_interface>
+      <state_interface name="position"/>
+      <state_interface name="velocity"/>
+      <param name="node_id">10</param>
     </joint>
     <!-- <joint name="br_m1_s1">

Commit message: Hardware BR leg is now working

File: description/ros2_control.xacro (robot description, xacro)
@@ -19,4 +19,11 @@
       <state_interface name="velocity"/>
       <param name="node_id">10</param>
+    </joint>
+    <joint name="br_l4_l3">
+      <command_interface name="position">
+      </command_interface>
+      <state_interface name="position"/>
+      <state_interface name="velocity"/>
+      <param name="node_id">11</param>
     </joint>
     <!-- <joint name="br_m1_s1">

Commit message: BL and BR legs working

File: description/ros2_control.xacro (robot description, xacro)
@@ -26,4 +26,25 @@
       <state_interface name="velocity"/>
       <param name="node_id">11</param>
+    </joint>
+    <joint name="bl_m1_s1">
+      <command_interface name="position">
+      </command_interface>
+      <state_interface name="position"/>
+      <state_interface name="velocity"/>
+      <param name="node_id">6</param>
+    </joint>
+    <joint name="bl_m2_s2">
+      <command_interface name="position">
+      </command_interface>
+      <state_interface name="position"/>
+      <state_interface name="velocity"/>
+      <param name="node_id">7</param>
+    </joint>
+    <joint name="bl_l4_l3">
+      <command_interface name="position">
+      </command_interface>
+      <state_interface name="position"/>
+      <state_interface name="velocity"/>
+      <param name="node_id">8</param>
     </joint>
     <!-- <joint name="br_m1_s1">

Commit message: added missing joint controllers

File: description/ros2_control.xacro (robot description, xacro)
@@ -6,24 +6,45 @@
       <param name="can">can0</param>
     </hardware>
-    <joint name="br_m1_s1">
+    <joint name="fl_m1_s1">
       <command_interface name="position">
       </command_interface>
       <state_interface name="position"/>
       <state_interface name="velocity"/>
-      <param name="node_id">9</param>
+      <param name="node_id">0</param>
     </joint>
-    <joint name="br_m2_s2">
+    <joint name="fl_m2_s2">
       <command_interface name="position">
       </command_interface>
       <state_interface name="position"/>
       <state_interface name="velocity"/>
-      <param name="node_id">10</param>
+      <param name="node_id">1</param>
     </joint>
-    <joint name="br_l4_l3">
+    <joint name="fl_l4_l3">
       <command_interface name="position">
       </command_interface>
       <state_interface name="position"/>
       <state_interface name="velocity"/>
-      <param name="node_id">11</param>
+      <param name="node_id">2</param>
+    </joint>
+    <joint name="fr_m1_s1">
+      <command_interface name="position">
+      </command_interface>
+      <state_interface name="position"/>
+      <state_interface name="velocity"/>
+      <param name="node_id">3</param>
+    </joint>
+    <joint name="fr_m2_s2">
+      <command_interface name="position">
+      </command_interface>
+      <state_interface name="position"/>
+      <state_interface name="velocity"/>
+      <param name="node_id">4</param>
+    </joint>
+    <joint name="fr_l4_s3">
+      <command_interface name="position">
+      </command_interface>
+      <state_interface name="position"/>
+      <state_interface name="velocity"/>
+      <param name="node_id">5</param>
     </joint>
     <joint name="bl_m1_s1">
@@ -47,4 +68,25 @@
       <state_interface name="velocity"/>
       <param name="node_id">8</param>
+    </joint>
+    <joint name="br_m1_s1">
+      <command_interface name="position">
+      </command_interface>
+      <state_interface name="position"/>
+      <state_interface name="velocity"/>
+      <param name="node_id">9</param>
+    </joint>
+    <joint name="br_m2_s2">
+      <command_interface name="position">
+      </command_interface>
+      <state_interface name="position"/>
+      <state_interface name="velocity"/>
+      <param name="node_id">10</param>
+    </joint>
+    <joint name="br_l4_l3">
+      <command_interface name="position">
+      </command_interface>
+      <state_interface name="position"/>
+      <state_interface name="velocity"/>
+      <param name="node_id">11</param>
     </joint>
     <!-- <joint name="br_m1_s1">

Commit message: fixed type

File: description/ros2_control.xacro (robot description, xacro)
@@ -41,5 +41,5 @@
       <param name="node_id">4</param>
     </joint>
-    <joint name="fr_l4_s3">
+    <joint name="fr_l4_l3">
       <command_interface name="position">
       </command_interface>

Commit message: changed control xacro file

File: description/ros2_control.xacro (robot description, xacro)
@@ -90,76 +90,4 @@
       <param name="node_id">11</param>
     </joint>
-    <!-- <joint name="br_m1_s1">
-      <command_interface name="position">
-      </command_interface>
-      <state_interface name="position"/>
-      <state_interface name="velocity"/>
-    </joint>
-    <joint name="br_m2_s2">
-      <command_interface name="position">
-      </command_interface>
-      <state_interface name="position"/>
-      <state_interface name="velocity"/>
-    </joint>
-    <joint name="br_m3_s3">
-      <command_interface name="position">
-      </command_interface>
-      <state_interface name="position"/>
-      <state_interface name="velocity"/>
-    </joint>
-    <joint name="bl_m1_s1">
-      <command_interface name="position">
-      </command_interface>
-      <state_interface name="position"/>
-      <state_interface name="velocity"/>
-    </joint>
-    <joint name="bl_m2_s2">
-      <command_interface name="position">
-      </command_interface>
-      <state_interface name="position"/>
-      <state_interface name="velocity"/>
-    </joint>
-    <joint name="bl_m3_s3">
-      <command_interface name="position">
-      </command_interface>
-      <state_interface name="position"/>
-      <state_interface name="velocity"/>
-    </joint>
-    <joint name="fr_m1_s1">
-      <command_interface name="position">
-      </command_interface>
-      <state_interface name="position"/>
-      <state_interface name="velocity"/>
-    </joint>
-    <joint name="fr_m2_s2">
-      <command_interface name="position">
-      </command_interface>
-      <state_interface name="position"/>
-      <state_interface name="velocity"/>
-    </joint>
-    <joint name="fr_m3_s3">
-      <command_interface name="position">
-      </command_interface>
-      <state_interface name="position"/>
-      <state_interface name="velocity"/>
-    </joint>
-    <joint name="fl_m1_s1">
-      <command_interface name="position">
-      </command_interface>
-      <state_interface name="position"/>
-      <state_interface name="velocity"/>
-    </joint>
-    <joint name="fl_m2_s2">
-      <command_interface name="position">
-      </command_interface>
-      <state_interface name="position"/>
-      <state_interface name="velocity"/>
-    </joint>
-    <joint name="fl_m3_s3">
-      <command_interface name="position">
-      </command_interface>
-      <state_interface name="position"/>
-      <state_interface name="velocity"/>
-    </joint> -->
   </ros2_control>
 </robot>
