Commit message: fixed arm to ground

File: description/quadro.xacro (robot description, xacro)
@@ -7,4 +7,5 @@
   <xacro:include filename="$(find quadro)/description/quadro.gazebo" />
 </xacro:if>
+<link name="world"></link>
 <link name="base_link">
   <inertial>
@@ -87,4 +88,9 @@
   </collision>
 </link>
+<joint name="base_joint" type="fixed">
+    <origin xyz="0.0 0.0 -0.07" rpy="0 0 0"/>
+    <parent link="world"/>
+    <child link="base_link"/>
+</joint>
 <joint name="BR1" type="continuous">
   <origin xyz="-0.000251 7e-06 0.0365" rpy="0 0 0"/>
@@ -92,5 +98,5 @@
   <child link="link_1_1"/>
   <axis xyz="0.0 0.0 -1.0"/>
-  <limit effort="12" velocity="30" lower="-12.565" upper="12.565"/>
+  <limit effort="12" velocity="2" lower="-12.565" upper="12.565"/>
 </joint>
 <joint name="BR2" type="continuous">
@@ -99,5 +105,5 @@
   <child link="link_2_1"/>
   <axis xyz="-1.0 0.0 0.0"/>
-  <limit effort="12" velocity="30" lower="-12.565" upper="12.565"/>
+  <limit effort="12" velocity="2" lower="-12.565" upper="12.565"/>
 </joint>
 <joint name="BR3" type="continuous">
@@ -106,5 +112,5 @@
   <child link="link_3_1"/>
   <axis xyz="-1.0 0.0 0.0"/>
-  <limit effort="12" velocity="30" lower="-12.565" upper="12.565"/>
+  <limit effort="12" velocity="2" lower="-12.565" upper="12.565"/>
 </joint>
 </robot>

Commit message: 2 dof mode workd

File: description/quadro.xacro (robot description, xacro)
@@ -1,5 +1,5 @@
 <?xml version="1.0" ?>
 <robot name="quadro" xmlns:xacro="http://www.ros.org/wiki/xacro">
-<xacro:arg name="sim_mode" default="true"/>
+<xacro:arg name="sim_mode" default="false"/>
 <xacro:include filename="$(find quadro)/description/materials.xacro" />
 <!-- <xacro:include filename="$(find quadro)/description/quadro.trans" /> -->
@@ -7,4 +7,7 @@
   <xacro:include filename="$(find quadro)/description/quadro.gazebo" />
 </xacro:if>
+<xacro:unless value="$(arg sim_mode)">
+  <xacro:include filename="$(find quadro)/description/ros2_control.xacro" />
+</xacro:unless>
 <link name="world"></link>
 <link name="base_link">
@@ -98,5 +101,5 @@
   <child link="link_1_1"/>
   <axis xyz="0.0 0.0 -1.0"/>
-  <limit effort="12" velocity="2" lower="-12.565" upper="12.565"/>
+  <limit effort="12" velocity="2" lower="-1.57" upper="1.57"/>
 </joint>
 <joint name="BR2" type="continuous">
@@ -105,5 +108,5 @@
   <child link="link_2_1"/>
   <axis xyz="-1.0 0.0 0.0"/>
-  <limit effort="12" velocity="2" lower="-12.565" upper="12.565"/>
+  <limit effort="120" velocity="4" lower="0.0" upper="1.20"/>
 </joint>
 <joint name="BR3" type="continuous">
@@ -112,5 +115,5 @@
   <child link="link_3_1"/>
   <axis xyz="-1.0 0.0 0.0"/>
-  <limit effort="12" velocity="2" lower="-12.565" upper="12.565"/>
+  <limit effort="120" velocity="4" lower="0.0" upper="1.20"/>
 </joint>
 </robot>

Commit message: first hardware integration tests

File: description/quadro.xacro (robot description, xacro)
@@ -430,5 +430,5 @@
     <parent link="shaft_2"/>
     <child link="shaft_3"/>
-    <axis xyz="0 0 -1"/>
+    <axis xyz="0 0 1"/>
     <limit effort="10" velocity="12" lower="-3.14" upper="3.14"/>
     <joint_properties friction="0.5"/>
@@ -512,5 +512,5 @@
     <parent link="shaft_2"/>
     <child link="lin_4_r"/>
-    <axis xyz="0 0 -1"/>
+    <axis xyz="0 0 1"/>
     <limit effort="10" velocity="12" lower="-3.14" upper="3.14"/>
     <joint_properties friction="0.5"/>
@@ -521,5 +521,5 @@
     <parent link="shaft"/>
     <child link="shaft_2"/>
-    <axis xyz="0 0 -1"/>
+    <axis xyz="0 0 1"/>
     <limit effort="10" velocity="12" lower="-3.14" upper="3.14"/>
     <joint_properties friction="0.5"/>
@@ -530,5 +530,5 @@
     <parent link="back_plate"/>
     <child link="shaft"/>
-    <axis xyz="0 0 -1"/>
+    <axis xyz="0 0 1"/>
     <limit effort="10" velocity="12" lower="-3.14" upper="3.14"/>
     <joint_properties friction="0.5"/>
@@ -739,5 +739,5 @@
     <parent link="shaft_5"/>
     <child link="shaft_6"/>
-    <axis xyz="0 0 -1"/>
+    <axis xyz="0 0 1"/>
     <limit effort="10" velocity="12" lower="-3.14" upper="3.14"/>
     <joint_properties friction="0.5"/>
@@ -821,5 +821,5 @@
     <parent link="shaft_5"/>
     <child link="lin_4_l"/>
-    <axis xyz="0 0 -1"/>
+    <axis xyz="0 0 1"/>
     <limit effort="10" velocity="12" lower="-3.14" upper="3.14"/>
     <joint_properties friction="0.5"/>
@@ -830,5 +830,5 @@
     <parent link="shaft_4"/>
     <child link="shaft_5"/>
-    <axis xyz="0 0 -1"/>
+    <axis xyz="0 0 1"/>
     <limit effort="10" velocity="12" lower="-3.14" upper="3.14"/>
     <joint_properties friction="0.5"/>
@@ -839,5 +839,5 @@
     <parent link="back_plate"/>
     <child link="shaft_4"/>
-    <axis xyz="0 0 -1"/>
+    <axis xyz="0 0 1"/>
     <limit effort="10" velocity="12" lower="-3.14" upper="3.14"/>
     <joint_properties friction="0.5"/>
@@ -1048,5 +1048,5 @@
     <parent link="shaft_8"/>
     <child link="shaft_9"/>
-    <axis xyz="0 0 -1"/>
+    <axis xyz="0 0 1"/>
     <limit effort="10" velocity="12" lower="-3.14" upper="3.14"/>
     <joint_properties friction="0.5"/>
@@ -1130,5 +1130,5 @@
     <parent link="shaft_8"/>
     <child link="lin_4_r_2"/>
-    <axis xyz="0 0 -1"/>
+    <axis xyz="0 0 1"/>
     <limit effort="10" velocity="12" lower="-3.14" upper="3.14"/>
     <joint_properties friction="0.5"/>
@@ -1139,5 +1139,5 @@
     <parent link="shaft_7"/>
     <child link="shaft_8"/>
-    <axis xyz="0 0 -1"/>
+    <axis xyz="0 0 1"/>
     <limit effort="10" velocity="12" lower="-3.14" upper="3.14"/>
     <joint_properties friction="0.5"/>
@@ -1148,5 +1148,5 @@
     <parent link="back_plate"/>
     <child link="shaft_7"/>
-    <axis xyz="0 0 -1"/>
+    <axis xyz="0 0 1"/>
     <limit effort="10" velocity="12" lower="-3.14" upper="3.14"/>
     <joint_properties friction="0.5"/>
@@ -1357,5 +1357,5 @@
     <parent link="motor_2"/>
     <child link="shaft_10"/>
-    <axis xyz="0 0 -1"/>
+    <axis xyz="0 0 1"/>
     <limit effort="10" velocity="12" lower="-3.14" upper="3.14"/>
     <joint_properties friction="0.5"/>
@@ -1439,5 +1439,5 @@
     <parent link="motor_2"/>
     <child link="lin_4_l_2"/>
-    <axis xyz="0 0 -1"/>
+    <axis xyz="0 0 1"/>
     <limit effort="10" velocity="12" lower="-3.14" upper="3.14"/>
     <joint_properties friction="0.5"/>
@@ -1448,5 +1448,5 @@
     <parent link="motor"/>
     <child link="motor_2"/>
-    <axis xyz="0 0 -1"/>
+    <axis xyz="0 0 1"/>
     <limit effort="10" velocity="12" lower="-3.14" upper="3.14"/>
     <joint_properties friction="0.5"/>
@@ -1457,5 +1457,5 @@
     <parent link="back_plate"/>
     <child link="motor"/>
-    <axis xyz="0 0 -1"/>
+    <axis xyz="0 0 1"/>
     <limit effort="10" velocity="12" lower="-3.14" upper="3.14"/>
     <joint_properties friction="0.5"/>
