Commit message: added v2 simulation design

File: description/quadro.xacro (robot description, xacro)
@@ -5,5 +5,5 @@
 <!-- <xacro:include filename="$(find quadro)/description/quadro.trans" /> -->
 <xacro:if value="$(arg sim_mode)">
-  <xacro:include filename="$(find quadro)/description/quadro.gazebo" />
+  <xacro:include filename="$(find quadro)/description/robot.gazebo" />
 </xacro:if>
 <xacro:unless value="$(arg sim_mode)">
@@ -12,7 +12,7 @@
   <link name="back_plate">
     <inertial>
-      <origin xyz="-0.139034 0.00943483 -0.0243213" rpy="0 0 0"/>
-      <mass value="2.38325"/>
-      <inertia ixx="0.0204343" ixy="-3.21203e-05" ixz="6.24877e-20" iyy="0.00715196" iyz="-3.89899e-19" izz="0.0254162"/>
+      <origin xyz="-0.139034 0.0124348 -0.00910543" rpy="0 0 0"/>
+      <mass value="1.72721"/>
+      <inertia ixx="0.0212545" ixy="-3.30055e-05" ixz="-6.76645e-13" iyy="0.00654795" iyz="1.86986e-13" izz="0.0255793"/>
     </inertial>
     <!-- Part back_stop -->
@@ -34,5 +34,5 @@
     <!-- Part side_pipe -->
     <visual>
-      <origin xyz="-0.0083688 0.0999348 -0.058441" rpy="0 -0 0"/>
+      <origin xyz="-0.286981 0.105935 -0.058441" rpy="0 -0 0"/>
       <geometry>
         <mesh filename="file://$(find quadro)/description/assets/side_pipe.stl"/>
@@ -43,12 +43,28 @@
     </visual>
     <collision>
-      <origin xyz="-0.0083688 0.0999348 -0.058441" rpy="0 -0 0"/>
+      <origin xyz="-0.286981 0.105935 -0.058441" rpy="0 -0 0"/>
       <geometry>
         <mesh filename="file://$(find quadro)/description/assets/side_pipe.stl"/>
       </geometry>
     </collision>
+    <!-- Part side_cover -->
+    <visual>
+      <origin xyz="-0.139034 -0.0810652 -0.058441" rpy="2.4928e-28 -8.23912e-18 -3.14159"/>
+      <geometry>
+        <mesh filename="file://$(find quadro)/description/assets/side_cover.stl"/>
+      </geometry>
+      <material name="side_cover_material">
+        <color rgba="0.647059 0.647059 0.647059 1"/>
+      </material>
+    </visual>
+    <collision>
+      <origin xyz="-0.139034 -0.0810652 -0.058441" rpy="2.4928e-28 -8.23912e-18 -3.14159"/>
+      <geometry>
+        <mesh filename="file://$(find quadro)/description/assets/side_cover.stl"/>
+      </geometry>
+    </collision>
     <!-- Part back_plate -->
     <visual>
-      <origin xyz="-0.139034 0.0999348 -0.058441" rpy="0 -0 0"/>
+      <origin xyz="-0.139034 0.105935 -0.058441" rpy="-3.9443e-31 6.56859e-46 -1.79651e-46"/>
       <geometry>
         <mesh filename="file://$(find quadro)/description/assets/back_plate.stl"/>
@@ -59,28 +75,12 @@
     </visual>
     <collision>
-      <origin xyz="-0.139034 0.0999348 -0.058441" rpy="0 -0 0"/>
+      <origin xyz="-0.139034 0.105935 -0.058441" rpy="-3.9443e-31 6.56859e-46 -1.79651e-46"/>
       <geometry>
         <mesh filename="file://$(find quadro)/description/assets/back_plate.stl"/>
       </geometry>
     </collision>
-    <!-- Part battery -->
-    <visual>
-      <origin xyz="-0.0725337 -0.0125652 -0.028441" rpy="0 -6.12323e-17 1.5708"/>
-      <geometry>
-        <mesh filename="file://$(find quadro)/description/assets/battery.stl"/>
-      </geometry>
-      <material name="battery_material">
-        <color rgba="0.768627 0.886275 0.952941 1"/>
-      </material>
-    </visual>
-    <collision>
-      <origin xyz="-0.0725337 -0.0125652 -0.028441" rpy="0 -6.12323e-17 1.5708"/>
-      <geometry>
-        <mesh filename="file://$(find quadro)/description/assets/battery.stl"/>
-      </geometry>
-    </collision>
     <!-- Part motor -->
     <visual>
-      <origin xyz="-0.194034 -0.0920652 -0.023441" rpy="3.14159 5.95406e-36 -1.5708"/>
+      <origin xyz="-0.194034 -0.0920652 -0.00844105" rpy="3.14159 5.95406e-36 -1.5708"/>
       <geometry>
         <mesh filename="file://$(find quadro)/description/assets/motor.stl"/>
@@ -91,12 +91,28 @@
     </visual>
     <collision>
-      <origin xyz="-0.194034 -0.0920652 -0.023441" rpy="3.14159 5.95406e-36 -1.5708"/>
-      <geometry>
-        <mesh filename="file://$(find quadro)/description/assets/motor.stl"/>
+      <origin xyz="-0.194034 -0.0920652 -0.00844105" rpy="3.14159 5.95406e-36 -1.5708"/>
+      <geometry>
+        <mesh filename="file://$(find quadro)/description/assets/motor.stl"/>
+      </geometry>
+    </collision>
+    <!-- Part side_cover_2 -->
+    <visual>
+      <origin xyz="-0.139034 0.105935 -0.058441" rpy="0 -8.23912e-18 2.00179e-32"/>
+      <geometry>
+        <mesh filename="file://$(find quadro)/description/assets/side_cover.stl"/>
+      </geometry>
+      <material name="side_cover_2_material">
+        <color rgba="0.647059 0.647059 0.647059 1"/>
+      </material>
+    </visual>
+    <collision>
+      <origin xyz="-0.139034 0.105935 -0.058441" rpy="0 -8.23912e-18 2.00179e-32"/>
+      <geometry>
+        <mesh filename="file://$(find quadro)/description/assets/side_cover.stl"/>
       </geometry>
     </collision>
     <!-- Part motor_2 -->
     <visual>
-      <origin xyz="-0.194034 0.110935 -0.023441" rpy="3.14159 5.95406e-36 1.5708"/>
+      <origin xyz="-0.194034 0.116935 -0.00844105" rpy="-3.14159 7.88861e-31 1.5708"/>
       <geometry>
         <mesh filename="file://$(find quadro)/description/assets/motor.stl"/>
@@ -107,5 +123,5 @@
     </visual>
     <collision>
-      <origin xyz="-0.194034 0.110935 -0.023441" rpy="3.14159 5.95406e-36 1.5708"/>
+      <origin xyz="-0.194034 0.116935 -0.00844105" rpy="-3.14159 7.88861e-31 1.5708"/>
       <geometry>
         <mesh filename="file://$(find quadro)/description/assets/motor.stl"/>
@@ -114,5 +130,5 @@
     <!-- Part motor_3 -->
     <visual>
-      <origin xyz="-0.0840337 -0.0920652 -0.023441" rpy="3.14159 5.95406e-36 -1.5708"/>
+      <origin xyz="-0.0840337 -0.0920652 -0.00844105" rpy="3.14159 5.95406e-36 -1.5708"/>
       <geometry>
         <mesh filename="file://$(find quadro)/description/assets/motor.stl"/>
@@ -123,12 +139,28 @@
     </visual>
     <collision>
-      <origin xyz="-0.0840337 -0.0920652 -0.023441" rpy="3.14159 5.95406e-36 -1.5708"/>
-      <geometry>
-        <mesh filename="file://$(find quadro)/description/assets/motor.stl"/>
+      <origin xyz="-0.0840337 -0.0920652 -0.00844105" rpy="3.14159 5.95406e-36 -1.5708"/>
+      <geometry>
+        <mesh filename="file://$(find quadro)/description/assets/motor.stl"/>
+      </geometry>
+    </collision>
+    <!-- Part bot_pipe_half -->
+    <visual>
+      <origin xyz="-0.139034 0.439935 -0.058441" rpy="3.14159 -0 0"/>
+      <geometry>
+        <mesh filename="file://$(find quadro)/description/assets/bot_pipe_half.stl"/>
+      </geometry>
+      <material name="bot_pipe_half_material">
+        <color rgba="0.972549 0.529412 0.00392157 1"/>
+      </material>
+    </visual>
+    <collision>
+      <origin xyz="-0.139034 0.439935 -0.058441" rpy="3.14159 -0 0"/>
+      <geometry>
+        <mesh filename="file://$(find quadro)/description/assets/bot_pipe_half.stl"/>
       </geometry>
     </collision>
     <!-- Part side_pipe_2 -->
     <visual>
-      <origin xyz="-0.139034 -0.0810652 0.0614484" rpy="3.14159 -0 0"/>
+      <origin xyz="-0.139034 -0.0810652 0.095559" rpy="3.14159 -0 0"/>
       <geometry>
         <mesh filename="file://$(find quadro)/description/assets/side_pipe.stl"/>
@@ -139,5 +171,5 @@
     </visual>
     <collision>
-      <origin xyz="-0.139034 -0.0810652 0.0614484" rpy="3.14159 -0 0"/>
+      <origin xyz="-0.139034 -0.0810652 0.095559" rpy="3.14159 -0 0"/>
       <geometry>
         <mesh filename="file://$(find quadro)/description/assets/side_pipe.stl"/>
@@ -146,5 +178,5 @@
     <!-- Part motor_4 -->
     <visual>
-      <origin xyz="-0.0840337 0.110935 -0.023441" rpy="3.14159 5.95406e-36 1.5708"/>
+      <origin xyz="-0.0840337 0.116935 -0.00844105" rpy="-3.14159 7.88861e-31 1.5708"/>
       <geometry>
         <mesh filename="file://$(find quadro)/description/assets/motor.stl"/>
@@ -155,5 +187,5 @@
     </visual>
     <collision>
-      <origin xyz="-0.0840337 0.110935 -0.023441" rpy="3.14159 5.95406e-36 1.5708"/>
+      <origin xyz="-0.0840337 0.116935 -0.00844105" rpy="-3.14159 7.88861e-31 1.5708"/>
       <geometry>
         <mesh filename="file://$(find quadro)/description/assets/motor.stl"/>
@@ -162,5 +194,5 @@
     <!-- Part back_stop_2 -->
     <visual>
-      <origin xyz="-0.139034 0.0520348 -0.058441" rpy="0 -0 3.14159"/>
+      <origin xyz="-0.139034 0.0580348 -0.058441" rpy="0 -0 -3.14159"/>
       <geometry>
         <mesh filename="file://$(find quadro)/description/assets/back_stop.stl"/>
@@ -171,5 +203,5 @@
     </visual>
     <collision>
-      <origin xyz="-0.139034 0.0520348 -0.058441" rpy="0 -0 3.14159"/>
+      <origin xyz="-0.139034 0.0580348 -0.058441" rpy="0 -0 -3.14159"/>
       <geometry>
         <mesh filename="file://$(find quadro)/description/assets/back_stop.stl"/>
@@ -192,34 +224,50 @@
       </geometry>
     </collision>
-    <!-- Part main_pipe -->
-    <visual>
-      <origin xyz="-0.139034 -0.133065 -0.058441" rpy="0 -0 0"/>
-      <geometry>
-        <mesh filename="file://$(find quadro)/description/assets/main_pipe.stl"/>
-      </geometry>
-      <material name="main_pipe_material">
-        <color rgba="0 0 0 1"/>
-      </material>
-    </visual>
-    <collision>
-      <origin xyz="-0.139034 -0.133065 -0.058441" rpy="0 -0 0"/>
-      <geometry>
-        <mesh filename="file://$(find quadro)/description/assets/main_pipe.stl"/>
-      </geometry>
-    </collision>
-    <!-- Part battery_2 -->
-    <visual>
-      <origin xyz="-0.205534 -0.0125652 -0.028441" rpy="3.14159 -6.12323e-17 1.5708"/>
-      <geometry>
-        <mesh filename="file://$(find quadro)/description/assets/battery.stl"/>
-      </geometry>
-      <material name="battery_2_material">
-        <color rgba="0.768627 0.886275 0.952941 1"/>
-      </material>
-    </visual>
-    <collision>
-      <origin xyz="-0.205534 -0.0125652 -0.028441" rpy="3.14159 -6.12323e-17 1.5708"/>
-      <geometry>
-        <mesh filename="file://$(find quadro)/description/assets/battery.stl"/>
+    <!-- Part bot_pipe_half_2 -->
+    <visual>
+      <origin xyz="-0.139034 -0.415065 -0.058441" rpy="0 -0 0"/>
+      <geometry>
+        <mesh filename="file://$(find quadro)/description/assets/bot_pipe_half.stl"/>
+      </geometry>
+      <material name="bot_pipe_half_2_material">
+        <color rgba="0.972549 0.529412 0.00392157 1"/>
+      </material>
+    </visual>
+    <collision>
+      <origin xyz="-0.139034 -0.415065 -0.058441" rpy="0 -0 0"/>
+      <geometry>
+        <mesh filename="file://$(find quadro)/description/assets/bot_pipe_half.stl"/>
+      </geometry>
+    </collision>
+    <!-- Part mid_clamp -->
+    <visual>
+      <origin xyz="-0.139034 0.245535 -0.058441" rpy="0 -0 0"/>
+      <geometry>
+        <mesh filename="file://$(find quadro)/description/assets/mid_clamp.stl"/>
+      </geometry>
+      <material name="mid_clamp_material">
+        <color rgba="1 0.756863 0.054902 1"/>
+      </material>
+    </visual>
+    <collision>
+      <origin xyz="-0.139034 0.245535 -0.058441" rpy="0 -0 0"/>
+      <geometry>
+        <mesh filename="file://$(find quadro)/description/assets/mid_clamp.stl"/>
+      </geometry>
+    </collision>
+    <!-- Part pierdolnik -->
+    <visual>
+      <origin xyz="-0.0467776 0.0689348 -0.136744" rpy="2.1209e-41 -1.5708 0"/>
+      <geometry>
+        <mesh filename="file://$(find quadro)/description/assets/pierdolnik.stl"/>
+      </geometry>
+      <material name="pierdolnik_material">
+        <color rgba="0.980392 0.713725 0.00392157 1"/>
+      </material>
+    </visual>
+    <collision>
+      <origin xyz="-0.0467776 0.0689348 -0.136744" rpy="2.1209e-41 -1.5708 0"/>
+      <geometry>
+        <mesh filename="file://$(find quadro)/description/assets/pierdolnik.stl"/>
       </geometry>
     </collision>
@@ -228,20 +276,20 @@
   <link name="shaft">
     <inertial>
-      <origin xyz="-0.00743033 0.00365203 -0.0538481" rpy="0 0 0"/>
-      <mass value="0.500834"/>
-      <inertia ixx="0.000715416" ixy="-4.87254e-05" ixz="-3.36343e-05" iyy="0.000667976" iyz="1.74582e-05" izz="0.000280763"/>
+      <origin xyz="-0.00615624 0.00516896 -0.0539841" rpy="0 0 0"/>
+      <mass value="0.498148"/>
+      <inertia ixx="0.000680513" ixy="-5.35146e-05" ixz="-2.97443e-05" iyy="0.000689619" iyz="2.85044e-05" izz="0.000273018"/>
     </inertial>
     <!-- Part lin_1_support_br -->
     <visual>
-      <origin xyz="-0.0242487 0.014 -0.0735" rpy="1.0472 -1.5708 0"/>
+      <origin xyz="-0.019799 0.019799 -0.0735" rpy="0.785398 -1.5708 0"/>
       <geometry>
         <mesh filename="file://$(find quadro)/description/assets/lin_1_support_br.stl"/>
       </geometry>
       <material name="lin_1_support_br_material">
-        <color rgba="1 0.756863 0.054902 1"/>
-      </material>
-    </visual>
-    <collision>
-      <origin xyz="-0.0242487 0.014 -0.0735" rpy="1.0472 -1.5708 0"/>
+        <color rgba="0.901961 0.901961 0.901961 1"/>
+      </material>
+    </visual>
+    <collision>
+      <origin xyz="-0.019799 0.019799 -0.0735" rpy="0.785398 -1.5708 0"/>
       <geometry>
         <mesh filename="file://$(find quadro)/description/assets/lin_1_support_br.stl"/>
@@ -250,5 +298,5 @@
     <!-- Part motor_5 -->
     <visual>
-      <origin xyz="-0.0147224 0.0085 -0.0735" rpy="-1.5708 6.61824e-17 -0.523599"/>
+      <origin xyz="-0.0120208 0.0120208 -0.0735" rpy="-1.5708 4.94218e-17 -0.785398"/>
       <geometry>
         <mesh filename="file://$(find quadro)/description/assets/motor.stl"/>
@@ -259,5 +307,5 @@
     </visual>
     <collision>
-      <origin xyz="-0.0147224 0.0085 -0.0735" rpy="-1.5708 6.61824e-17 -0.523599"/>
+      <origin xyz="-0.0120208 0.0120208 -0.0735" rpy="-1.5708 4.94218e-17 -0.785398"/>
       <geometry>
         <mesh filename="file://$(find quadro)/description/assets/motor.stl"/>
@@ -284,43 +332,43 @@
   <link name="shaft_2">
     <inertial>
-      <origin xyz="0.0106548 -0.00501565 -0.0435875" rpy="0 0 0"/>
-      <mass value="0.551476"/>
-      <inertia ixx="0.000599797" ixy="0.000304448" ixz="0.000186335" iyy="0.00130385" iyz="-9.91623e-05" izz="0.00132343"/>
-    </inertial>
-    <!-- Part lin_3_bot_r -->
-    <visual>
-      <origin xyz="2.77556e-17 8.04912e-16 -0.0645" rpy="1.5708 -3.60822e-16 2.79253"/>
-      <geometry>
-        <mesh filename="file://$(find quadro)/description/assets/lin_3_bot_r.stl"/>
-      </geometry>
-      <material name="lin_3_bot_r_material">
-        <color rgba="1 0.756863 0.054902 1"/>
-      </material>
-    </visual>
-    <collision>
-      <origin xyz="2.77556e-17 8.04912e-16 -0.0645" rpy="1.5708 -3.60822e-16 2.79253"/>
-      <geometry>
-        <mesh filename="file://$(find quadro)/description/assets/lin_3_bot_r.stl"/>
-      </geometry>
-    </collision>
-    <!-- Part lin_3_top_r -->
-    <visual>
-      <origin xyz="2.77556e-17 8.04912e-16 -0.0645" rpy="1.5708 -2.77556e-16 2.79253"/>
-      <geometry>
-        <mesh filename="file://$(find quadro)/description/assets/lin_3_top_r.stl"/>
-      </geometry>
-      <material name="lin_3_top_r_material">
-        <color rgba="1 0.756863 0.054902 1"/>
-      </material>
-    </visual>
-    <collision>
-      <origin xyz="2.77556e-17 8.04912e-16 -0.0645" rpy="1.5708 -2.77556e-16 2.79253"/>
-      <geometry>
-        <mesh filename="file://$(find quadro)/description/assets/lin_3_top_r.stl"/>
+      <origin xyz="0.0151537 -0.00339527 -0.0487431" rpy="0 0 0"/>
+      <mass value="0.644469"/>
+      <inertia ixx="0.000638791" ixy="0.000110507" ixz="0.000284701" iyy="0.00153132" iyz="-7.36435e-05" izz="0.00136973"/>
+    </inertial>
+    <!-- Part bot_4 -->
+    <visual>
+      <origin xyz="-6.93889e-16 1.9984e-15 0.1275" rpy="-1.5708 6.93889e-16 -0.0872665"/>
+      <geometry>
+        <mesh filename="file://$(find quadro)/description/assets/bot_4.stl"/>
+      </geometry>
+      <material name="bot_4_material">
+        <color rgba="0.901961 0.901961 0.901961 1"/>
+      </material>
+    </visual>
+    <collision>
+      <origin xyz="-6.93889e-16 1.9984e-15 0.1275" rpy="-1.5708 6.93889e-16 -0.0872665"/>
+      <geometry>
+        <mesh filename="file://$(find quadro)/description/assets/bot_4.stl"/>
+      </geometry>
+    </collision>
+    <!-- Part top_r -->
+    <visual>
+      <origin xyz="-7.77156e-16 2.02616e-15 0.1275" rpy="-1.5708 5.48173e-16 -0.0872665"/>
+      <geometry>
+        <mesh filename="file://$(find quadro)/description/assets/top_r.stl"/>
+      </geometry>
+      <material name="top_r_material">
+        <color rgba="0.901961 0.901961 0.901961 1"/>
+      </material>
+    </visual>
+    <collision>
+      <origin xyz="-7.77156e-16 2.02616e-15 0.1275" rpy="-1.5708 5.48173e-16 -0.0872665"/>
+      <geometry>
+        <mesh filename="file://$(find quadro)/description/assets/top_r.stl"/>
       </geometry>
     </collision>
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