Commit message: some usd changes

File: description/quadro.xacro (robot description, xacro)
@@ -12,7 +12,7 @@
   <link name="back_plate">
     <inertial>
-      <origin xyz="-0.139034 0.0124348 -0.00910543" rpy="0 0 0"/>
-      <mass value="1.72721"/>
-      <inertia ixx="0.0212545" ixy="-3.30055e-05" ixz="-6.76645e-13" iyy="0.00654795" iyz="1.86986e-13" izz="0.0255793"/>
+      <origin xyz="-0.139034 0.00733582 -0.013731" rpy="0 0 0"/>
+      <mass value="2.59053"/>
+      <inertia ixx="0.0255846" ixy="-4.15339e-05" ixz="-1.35405e-12" iyy="0.00872593" iyz="-0.000207516" izz="0.0313278"/>
     </inertial>
     <!-- Part back_stop -->
@@ -80,4 +80,20 @@
       </geometry>
     </collision>
+    <!-- Part battery -->
+    <visual>
+      <origin xyz="-0.0725337 -0.0315652 -0.029441" rpy="0 -6.12323e-17 1.5708"/>
+      <geometry>
+        <mesh filename="file://$(find quadro)/description/assets/battery.stl"/>
+      </geometry>
+      <material name="battery_material">
+        <color rgba="0.768627 0.886275 0.952941 1"/>
+      </material>
+    </visual>
+    <collision>
+      <origin xyz="-0.0725337 -0.0315652 -0.029441" rpy="0 -6.12323e-17 1.5708"/>
+      <geometry>
+        <mesh filename="file://$(find quadro)/description/assets/battery.stl"/>
+      </geometry>
+    </collision>
     <!-- Part motor -->
     <visual>
@@ -256,18 +272,18 @@
       </geometry>
     </collision>
-    <!-- Part pierdolnik -->
-    <visual>
-      <origin xyz="-0.0467776 0.0689348 -0.136744" rpy="2.1209e-41 -1.5708 0"/>
-      <geometry>
-        <mesh filename="file://$(find quadro)/description/assets/pierdolnik.stl"/>
-      </geometry>
-      <material name="pierdolnik_material">
-        <color rgba="0.980392 0.713725 0.00392157 1"/>
-      </material>
-    </visual>
-    <collision>
-      <origin xyz="-0.0467776 0.0689348 -0.136744" rpy="2.1209e-41 -1.5708 0"/>
-      <geometry>
-        <mesh filename="file://$(find quadro)/description/assets/pierdolnik.stl"/>
+    <!-- Part battery_2 -->
+    <visual>
+      <origin xyz="-0.205534 -0.0315652 -0.029441" rpy="3.14159 -0 1.5708"/>
+      <geometry>
+        <mesh filename="file://$(find quadro)/description/assets/battery.stl"/>
+      </geometry>
+      <material name="battery_2_material">
+        <color rgba="0.768627 0.886275 0.952941 1"/>
+      </material>
+    </visual>
+    <collision>
+      <origin xyz="-0.205534 -0.0315652 -0.029441" rpy="3.14159 -0 1.5708"/>
+      <geometry>
+        <mesh filename="file://$(find quadro)/description/assets/battery.stl"/>
       </geometry>
     </collision>
@@ -276,7 +292,7 @@
   <link name="shaft">
     <inertial>
-      <origin xyz="-0.00615624 0.00516896 -0.0539841" rpy="0 0 0"/>
-      <mass value="0.498148"/>
-      <inertia ixx="0.000680513" ixy="-5.35146e-05" ixz="-2.97443e-05" iyy="0.000689619" iyz="2.85044e-05" izz="0.000273018"/>
+      <origin xyz="-0.00474046 0.00407901 -0.0612986" rpy="0 0 0"/>
+      <mass value="0.452938"/>
+      <inertia ixx="0.000550761" ixy="-6.00381e-05" ixz="-1.13918e-05" iyy="0.00055728" iyz="1.18589e-05" izz="0.000239291"/>
     </inertial>
     <!-- Part lin_1_support_br -->
@@ -332,27 +348,27 @@
   <link name="shaft_2">
     <inertial>
-      <origin xyz="0.0151537 -0.00339527 -0.0487431" rpy="0 0 0"/>
-      <mass value="0.644469"/>
-      <inertia ixx="0.000638791" ixy="0.000110507" ixz="0.000284701" iyy="0.00153132" iyz="-7.36435e-05" izz="0.00136973"/>
-    </inertial>
-    <!-- Part bot_4 -->
-    <visual>
-      <origin xyz="-6.93889e-16 1.9984e-15 0.1275" rpy="-1.5708 6.93889e-16 -0.0872665"/>
-      <geometry>
-        <mesh filename="file://$(find quadro)/description/assets/bot_4.stl"/>
-      </geometry>
-      <material name="bot_4_material">
-        <color rgba="0.901961 0.901961 0.901961 1"/>
-      </material>
-    </visual>
-    <collision>
-      <origin xyz="-6.93889e-16 1.9984e-15 0.1275" rpy="-1.5708 6.93889e-16 -0.0872665"/>
-      <geometry>
-        <mesh filename="file://$(find quadro)/description/assets/bot_4.stl"/>
+      <origin xyz="0.00931177 -0.00187407 -0.0491985" rpy="0 0 0"/>
+      <mass value="0.524841"/>
+      <inertia ixx="0.000439148" ixy="6.14395e-05" ixz="0.000140002" iyy="0.000912333" iyz="-3.78102e-05" izz="0.000883052"/>
+    </inertial>
+    <!-- Part bot_r -->
+    <visual>
+      <origin xyz="5.55112e-16 3.60822e-16 0.1275" rpy="-1.5708 1.35308e-15 -0.0872665"/>
+      <geometry>
+        <mesh filename="file://$(find quadro)/description/assets/bot_r.stl"/>
+      </geometry>
+      <material name="bot_r_material">
+        <color rgba="0.901961 0.901961 0.901961 1"/>
+      </material>
+    </visual>
+    <collision>
+      <origin xyz="5.55112e-16 3.60822e-16 0.1275" rpy="-1.5708 1.35308e-15 -0.0872665"/>
+      <geometry>
+        <mesh filename="file://$(find quadro)/description/assets/bot_r.stl"/>
       </geometry>
     </collision>
     <!-- Part top_r -->
     <visual>
-      <origin xyz="-7.77156e-16 2.02616e-15 0.1275" rpy="-1.5708 5.48173e-16 -0.0872665"/>
+      <origin xyz="4.71845e-16 3.88578e-16 0.1275" rpy="-1.5708 1.20043e-15 -0.0872665"/>
       <geometry>
         <mesh filename="file://$(find quadro)/description/assets/top_r.stl"/>
@@ -363,5 +379,5 @@
     </visual>
     <collision>
-      <origin xyz="-7.77156e-16 2.02616e-15 0.1275" rpy="-1.5708 5.48173e-16 -0.0872665"/>
+      <origin xyz="4.71845e-16 3.88578e-16 0.1275" rpy="-1.5708 1.20043e-15 -0.0872665"/>
       <geometry>
         <mesh filename="file://$(find quadro)/description/assets/top_r.stl"/>
@@ -370,5 +386,5 @@
     <!-- Part shaft_2 -->
     <visual>
-      <origin xyz="0 -2.77556e-17 0.01" rpy="1.5708 1.5708 0"/>
+      <origin xyz="2.77556e-17 2.77556e-17 0.01" rpy="1.5708 1.5708 0"/>
       <geometry>
         <mesh filename="file://$(find quadro)/description/assets/shaft.stl"/>
@@ -379,5 +395,5 @@
     </visual>
     <collision>
-      <origin xyz="0 -2.77556e-17 0.01" rpy="1.5708 1.5708 0"/>
+      <origin xyz="2.77556e-17 2.77556e-17 0.01" rpy="1.5708 1.5708 0"/>
       <geometry>
         <mesh filename="file://$(find quadro)/description/assets/shaft.stl"/>
@@ -386,5 +402,5 @@
     <!-- Part lin_2_br -->
     <visual>
-      <origin xyz="-1.11022e-15 1.47105e-15 0.0305" rpy="-1.5708 -1.55431e-15 0.698132"/>
+      <origin xyz="8.32667e-17 0 0.0305" rpy="-1.5708 -2.33147e-15 0.698132"/>
       <geometry>
         <mesh filename="file://$(find quadro)/description/assets/lin_2_br.stl"/>
@@ -395,5 +411,5 @@
     </visual>
     <collision>
-      <origin xyz="-1.11022e-15 1.47105e-15 0.0305" rpy="-1.5708 -1.55431e-15 0.698132"/>
+      <origin xyz="8.32667e-17 0 0.0305" rpy="-1.5708 -2.33147e-15 0.698132"/>
       <geometry>
         <mesh filename="file://$(find quadro)/description/assets/lin_2_br.stl"/>
@@ -402,5 +418,5 @@
     <!-- Part motor_6 -->
     <visual>
-      <origin xyz="-1.13798e-15 1.33227e-15 -0.0395" rpy="0.872665 1.5708 0"/>
+      <origin xyz="2.77556e-17 -2.77556e-17 -0.0395" rpy="0.872665 1.5708 0"/>
       <geometry>
         <mesh filename="file://$(find quadro)/description/assets/motor.stl"/>
@@ -411,5 +427,5 @@
     </visual>
     <collision>
-      <origin xyz="-1.13798e-15 1.33227e-15 -0.0395" rpy="0.872665 1.5708 0"/>
+      <origin xyz="2.77556e-17 -2.77556e-17 -0.0395" rpy="0.872665 1.5708 0"/>
       <geometry>
         <mesh filename="file://$(find quadro)/description/assets/motor.stl"/>
@@ -420,7 +436,7 @@
   <link name="shaft_3">
     <inertial>
-      <origin xyz="0.00467702 0.00467702 -0.014107" rpy="0 0 0"/>
-      <mass value="0.152155"/>
-      <inertia ixx="4.49402e-05" ixy="-2.0502e-05" ixz="9.88665e-06" iyy="4.49402e-05" iyz="9.88665e-06" izz="6.45931e-05"/>
+      <origin xyz="0.00823991 0.00823991 -0.0152617" rpy="0 0 0"/>
+      <mass value="0.0992632"/>
+      <inertia ixx="3.95043e-05" ixy="-2.3154e-05" ixz="1.04189e-05" iyy="3.95043e-05" iyz="1.04189e-05" izz="6.07656e-05"/>
     </inertial>
     <!-- Part bearing -->
@@ -475,5 +491,5 @@
   <!-- Joint from shaft_2 to shaft_3 -->
   <joint name="br_m3_s3" type="revolute">
-    <origin xyz="-1.13798e-15 1.27676e-15 -0.0495" rpy="-2.27596e-15 -6.93889e-17 -0.226893"/>
+    <origin xyz="2.77556e-17 -2.77556e-17 -0.0495" rpy="-6.10623e-16 8.46545e-16 -0.226893"/>
     <parent link="shaft_2"/>
     <child link="shaft_3"/>
@@ -486,11 +502,11 @@
   <link name="l4_r">
     <inertial>
-      <origin xyz="0.00132696 -0.0488871 -0.00598393" rpy="0 0 0"/>
-      <mass value="0.128547"/>
-      <inertia ixx="0.00060149" ixy="-5.98605e-06" ixz="7.4372e-07" iyy="1.4027e-05" iyz="-4.69417e-06" izz="0.000610516"/>
+      <origin xyz="0.000903864 -0.036899 -0.00535524" rpy="0 0 0"/>
+      <mass value="0.0940232"/>
+      <inertia ixx="0.000523053" ixy="-1.96406e-06" ixz="4.23983e-07" iyy="8.81625e-06" iyz="-3.90493e-06" izz="0.000528442"/>
     </inertial>
     <!-- Part l4_r -->
     <visual>
-      <origin xyz="-0.16 0.002 0.192" rpy="-1.5708 -0 -5.55112e-17"/>
+      <origin xyz="-0.16 0.002 0.192" rpy="-1.5708 -0 -2.77556e-17"/>
       <geometry>
         <mesh filename="file://$(find quadro)/description/assets/l4_r.stl"/>
@@ -501,5 +517,5 @@
     </visual>
     <collision>
-      <origin xyz="-0.16 0.002 0.192" rpy="-1.5708 -0 -5.55112e-17"/>
+      <origin xyz="-0.16 0.002 0.192" rpy="-1.5708 -0 -2.77556e-17"/>
       <geometry>
         <mesh filename="file://$(find quadro)/description/assets/l4_r.stl"/>
@@ -508,5 +524,5 @@
     <!-- Part feet -->
     <visual>
-      <origin xyz="0.200014 0.04 -0.039" rpy="-1.5708 5.55112e-17 -2.41474e-15"/>
+      <origin xyz="0.200014 0.04 -0.039" rpy="-1.5708 -0 -2.44249e-15"/>
       <geometry>
         <mesh filename="file://$(find quadro)/description/assets/feet.stl"/>
@@ -517,5 +533,5 @@
     </visual>
     <collision>
-      <origin xyz="0.200014 0.04 -0.039" rpy="-1.5708 5.55112e-17 -2.41474e-15"/>
+      <origin xyz="0.200014 0.04 -0.039" rpy="-1.5708 -0 -2.44249e-15"/>
       <geometry>
         <mesh filename="file://$(find quadro)/description/assets/feet.stl"/>
@@ -524,5 +540,5 @@
     <!-- Part bearing_2 -->
     <visual>
-      <origin xyz="-5.55112e-17 0.055 -0.008" rpy="-1.5708 -1.11022e-16 0"/>
+      <origin xyz="5.55112e-17 0.055 -0.008" rpy="-1.5708 -1.11022e-16 2.77556e-17"/>
       <geometry>
         <mesh filename="file://$(find quadro)/description/assets/bearing.stl"/>
@@ -533,5 +549,5 @@
     </visual>
     <collision>
-      <origin xyz="-5.55112e-17 0.055 -0.008" rpy="-1.5708 -1.11022e-16 0"/>
+      <origin xyz="5.55112e-17 0.055 -0.008" rpy="-1.5708 -1.11022e-16 2.77556e-17"/>
       <geometry>
         <mesh filename="file://$(find quadro)/description/assets/bearing.stl"/>
@@ -540,5 +556,5 @@
     <!-- Part bearing_3 -->
     <visual>
-      <origin xyz="-1.11022e-16 0 -0.008" rpy="-1.5708 -5.55112e-17 0"/>
+      <origin xyz="1.11022e-16 2.77556e-17 -0.008" rpy="-1.5708 -5.55112e-17 0"/>
       <geometry>
         <mesh filename="file://$(find quadro)/description/assets/bearing.stl"/>
@@ -549,13 +565,28 @@
     </visual>
     <collision>
-      <origin xyz="-1.11022e-16 0 -0.008" rpy="-1.5708 -5.55112e-17 0"/>
-      <geometry>
-        <mesh filename="file://$(find quadro)/description/assets/bearing.stl"/>
-      </geometry>
-    </collision>
-  </link>
+      <origin xyz="1.11022e-16 2.77556e-17 -0.008" rpy="-1.5708 -5.55112e-17 0"/>
+      <geometry>
+        <mesh filename="file://$(find quadro)/description/assets/bearing.stl"/>
+      </geometry>
+    </collision>
+  </link>
+  <!-- Frame br_foot (dummy link + fixed joint) -->
+  <link name="br_foot">
+    <origin xyz="0 0 0" rpy="0 -0 0"/>
+    <inertial>
+      <origin xyz="0 0 0" rpy="0 0 0"/>
+      <mass value="1e-9"/>
+      <inertia ixx="0" ixy="0" ixz="0" iyy="0" iyz="0" izz="0"/>
+    </inertial>
+  </link>
+  <joint name="br_foot_frame" type="fixed">
+    <origin xyz="1.66533e-16 -0.165803 -0.004" rpy="-1.5708 -0 -2.44249e-15"/>
+    <parent link="l4_r"/>
+    <child link="br_foot"/>
+    <axis xyz="0 0 0"/>
+  </joint>
   <!-- Joint from shaft_2 to l4_r -->
   <joint name="br_l4_l3" type="revolute">
-    <origin xyz="0.159217 -0.0159373 -0.0735" rpy="-2.22045e-15 2.60902e-15 -1.01229"/>
+    <origin xyz="0.159217 -0.0159373 -0.0735" rpy="-1.72085e-15 4.38538e-15 -1.01229"/>
     <parent link="shaft_2"/>
     <child link="l4_r"/>
@@ -585,7 +616,7 @@
   <link name="shaft_4">
     <inertial>
-      <origin xyz="0.00614962 0.00518173 -0.0536475" rpy="0 0 0"/>
-      <mass value="0.498298"/>
-      <inertia ixx="0.000674129" ixy="5.36508e-05" ixz="3.04609e-05" iyy="0.000683037" iyz="2.79273e-05" izz="0.000273356"/>
+      <origin xyz="0.00473706 0.0040862 -0.0608763" rpy="0 0 0"/>
+      <mass value="0.453012"/>
+      <inertia ixx="0.000546146" ixy="6.01031e-05" ixz="1.17627e-05" iyy="0.000552555" iyz="1.15907e-05" izz="0.000239462"/>
     </inertial>
     <!-- Part shaft_4 -->
@@ -641,7 +672,7 @@
   <link name="shaft_5">
     <inertial>
-      <origin xyz="0.0112104 0.0105552 -0.0487431" rpy="0 0 0"/>
-      <mass value="0.644469"/>
-      <inertia ixx="0.000957084" ixy="-0.000442989" ixz="0.000209292" iyy="0.00121566" iyz="0.000206206" izz="0.00137236"/>
+      <origin xyz="0.00679431 0.00633758 -0.0491985" rpy="0 0 0"/>
+      <mass value="0.524841"/>
+      <inertia ixx="0.000610231" ixy="-0.000236595" ixz="0.000101861" iyy="0.000743295" iyz="0.00010283" izz="0.000885096"/>
     </inertial>
     <!-- Part lin_2_bl -->
@@ -729,7 +760,7 @@
   <link name="shaft_6">
     <inertial>
-      <origin xyz="-0.00467702 0.00467702 -0.014107" rpy="0 0 0"/>
-      <mass value="0.152155"/>
-      <inertia ixx="4.49402e-05" ixy="2.0502e-05" ixz="-9.88665e-06" iyy="4.49402e-05" iyz="9.88665e-06" izz="6.45931e-05"/>
+      <origin xyz="-0.00823991 0.00823991 -0.0152617" rpy="0 0 0"/>
+      <mass value="0.0992632"/>
+      <inertia ixx="3.95043e-05" ixy="2.3154e-05" ixz="-1.04189e-05" iyy="3.95043e-05" iyz="1.04189e-05" izz="6.07656e-05"/>
     </inertial>
     <!-- Part bearing_4 -->
@@ -795,7 +826,7 @@
   <link name="l4_l">
     <inertial>
-      <origin xyz="0.00132707 0.0488871 -0.00598393" rpy="0 0 0"/>
-      <mass value="0.128547"/>
-      <inertia ixx="0.00060149" ixy="5.98455e-06" ixz="7.43702e-07" iyy="1.40269e-05" iyz="4.69417e-06" izz="0.000610516"/>
+      <origin xyz="0.000904018 0.036899 -0.00535524" rpy="0 0 0"/>
+      <mass value="0.0940232"/>
+      <inertia ixx="0.000523053" ixy="1.96238e-06" ixz="4.23975e-07" iyy="8.81622e-06" iyz="3.90493e-06" izz="0.000528442"/>
     </inertial>
     <!-- Part bearing_5 -->
@@ -864,4 +895,19 @@
     </collision>
   </link>
+  <!-- Frame bl_foot (dummy link + fixed joint) -->
+  <link name="bl_foot">
+    <origin xyz="0 0 0" rpy="0 -0 0"/>
+    <inertial>
+      <origin xyz="0 0 0" rpy="0 0 0"/>
+      <mass value="1e-9"/>
+      <inertia ixx="0" ixy="0" ixz="0" iyy="0" iyz="0" izz="0"/>
+    </inertial>
+  </link>
+  <joint name="bl_foot_frame" type="fixed">
+    <origin xyz="-5.55112e-17 0.165803 -0.004" rpy="-1.5708 -1.66533e-16 -3.14159"/>
+    <parent link="l4_l"/>
+    <child link="bl_foot"/>
+    <axis xyz="0 0 0"/>
+  </joint>
   <!-- Joint from shaft_5 to l4_l -->
   <joint name="bl_l4_l3" type="revolute">
@@ -894,7 +940,7 @@
   <link name="shaft_7">
     <inertial>
-      <origin xyz="-0.00608141 -0.00524995 -0.0536475" rpy="0 0 0"/>
-      <mass value="0.498298"/>
-      <inertia ixx="0.000672811" ixy="5.36814e-05" ixz="-3.14816e-05" iyy="0.000684416" iyz="-2.69066e-05" izz="0.000273417"/>
+      <origin xyz="-0.00469968 -0.00412358 -0.0608763" rpy="0 0 0"/>
+      <mass value="0.453012"/>
+      <inertia ixx="0.000545527" ixy="6.01135e-05" ixz="-1.23936e-05" iyy="0.000553194" iyz="-1.09597e-05" izz="0.000239482"/>
     </inertial>
     <!-- Part lin_1_support_fr -->
@@ -950,7 +996,7 @@
   <link name="shaft_8">
     <inertial>
-      <origin xyz="0.0156244 -0.00329073 -0.0486585" rpy="0 0 0"/>
-      <mass value="0.64666"/>
-      <inertia ixx="0.000644429" ixy="0.000111011" ixz="0.000277194" iyy="0.00152296" iyz="-7.53778e-05" izz="0.00136428"/>
+      <origin xyz="0.00960955 -0.00201737 -0.0491732" rpy="0 0 0"/>
+      <mass value="0.525416"/>
+      <inertia ixx="0.000440202" ixy="6.05777e-05" ixz="0.000136109" iyy="0.000909648" iyz="-3.55951e-05" izz="0.000880794"/>
     </inertial>
     <!-- Part lin_2_fr -->
@@ -1018,11 +1064,11 @@
       </geometry>
     </collision>
-    <!-- Part bot_4_2 -->
+    <!-- Part bot_r_2 -->
     <visual>
       <origin xyz="8.32667e-17 1.11022e-16 0.1275" rpy="-1.5708 -9.02056e-17 -0.0872665"/>
       <geometry>
-        <mesh filename="file://$(find quadro)/description/assets/bot_4.stl"/>
-      </geometry>
-      <material name="bot_4_2_material">
+        <mesh filename="file://$(find quadro)/description/assets/bot_r.stl"/>
+      </geometry>
+      <material name="bot_r_2_material">
         <color rgba="0.901961 0.901961 0.901961 1"/>
       </material>
@@ -1031,5 +1077,5 @@
       <origin xyz="8.32667e-17 1.11022e-16 0.1275" rpy="-1.5708 -9.02056e-17 -0.0872665"/>
       <geometry>
-        <mesh filename="file://$(find quadro)/description/assets/bot_4.stl"/>
+        <mesh filename="file://$(find quadro)/description/assets/bot_r.stl"/>
       </geometry>
     </collision>
@@ -1038,7 +1084,7 @@
   <link name="shaft_9">
     <inertial>
-      <origin xyz="0.00467702 0.00467702 -0.014107" rpy="0 0 0"/>
-      <mass value="0.152155"/>
-      <inertia ixx="4.49402e-05" ixy="-2.0502e-05" ixz="9.88665e-06" iyy="4.49402e-05" iyz="9.88665e-06" izz="6.45931e-05"/>
+      <origin xyz="0.00823991 0.00823991 -0.0152617" rpy="0 0 0"/>
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
File: isaac_sim_files/quadro.urdf (robot description, URDF)
Before this commit: robot quadro, 17 links, 16 joints
Links:
- added link bl_foot, mass 1e-9
- added link br_foot, mass 1e-9
- added link fl_foot, mass 1e-9
- added link fr_foot, mass 1e-9
- link back_plate: mass 1.72721 -> 2.59053; geometry collision mesh filename=file:///home/rooteq/ros2_ws/install/quadro/share/quadro/des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; collision mesh filename=file:///home/rooteq/ros2_ws/install/quadro/share/quadro/des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
- link l4_l: mass 0.128547 -> 0.0940232
- link l4_l_2: mass 0.128547 -> 0.0940232
- link l4_r: mass 0.128547 -> 0.0940232
- link l4_r_2: mass 0.128547 -> 0.0940232
- link motor: mass 0.498148 -> 0.452937
- link motor_2: mass 0.64666 -> 0.525416
- link shaft: mass 0.498148 -> 0.452938
- link shaft_10: mass 0.152155 -> 0.0992632
- link shaft_2: mass 0.644469 -> 0.524841
- link shaft_3: mass 0.152155 -> 0.0992632
- link shaft_4: mass 0.498298 -> 0.453012
- link shaft_5: mass 0.644469 -> 0.524841
- link shaft_6: mass 0.152155 -> 0.0992632
- link shaft_7: mass 0.498298 -> 0.453012
- link shaft_8: mass 0.64666 -> 0.525416
- link shaft_9: mass 0.152155 -> 0.0992632
Joints:
- added joint bl_foot_frame: type fixed, parent l4_l, child bl_foot, origin xyz=-5.55112e-17 0.165803 -0.004 rpy=-1.5708 -1.66533e-16 -3.14159, axis 0 0 0
- added joint br_foot_frame: type fixed, parent l4_r, child br_foot, origin xyz=1.66533e-16 -0.165803 -0.004 rpy=-1.5708 -0 -2.44249e-15, axis 0 0 0
- added joint fl_foot_frame: type fixed, parent l4_l_2, child fl_foot, origin xyz=4.16334e-17 0.165803 -0.004 rpy=-1.5708 1.11022e-16 3.14159, axis 0 0 0
- added joint fr_foot_frame: type fixed, parent l4_r_2, child fr_foot, origin xyz=-8.32667e-17 -0.165803 -0.004 rpy=-1.5708 1.66533e-16 1.38778e-16, axis 0 0 0
- joint br_l4_l3: origin xyz=0.159217 -0.0159373 -0.0735 rpy=-2.22045e-15 2.60902e-15 -1.01229 -> xyz=0.159217 -0.0159373 -0.0735 rpy=-1.72085e-15 4.38538e-15 -1.01229
- joint br_m3_s3: origin xyz=-1.13798e-15 1.27676e-15 -0.0495 rpy=-2.27596e-15 -6.93889e-17 -0.226893 -> xyz=2.77556e-17 -2.77556e-17 -0.0495 rpy=-6.10623e-16 8.46545e-16 -0.226893
