Commit message: reinforcement learning setup works

File: isaac_sim_files/quadro.urdf (robot description, URDF)
Before this commit: robot quadro, 21 links, 20 joints
Links:
- removed link bl_foot
- removed link br_foot
- removed link fl_foot
- removed link fr_foot
- added link feet, mass 0.0122519; collision mesh filename=file:///home/rooteq/ros2_ws/install/quadro/share/quadro/des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; visual mesh filename=file:///home/rooteq/ros2_ws/install/quadro/share/quadro/des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
- added link feet_2, mass 0.0122519; collision mesh filename=file:///home/rooteq/ros2_ws/install/quadro/share/quadro/des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; visual mesh filename=file:///home/rooteq/ros2_ws/install/quadro/share/quadro/des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
- added link feet_3, mass 0.0122519; collision mesh filename=file:///home/rooteq/ros2_ws/install/quadro/share/quadro/des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; visual mesh filename=file:///home/rooteq/ros2_ws/install/quadro/share/quadro/des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
- added link feet_4, mass 0.0122519; collision mesh filename=file:///home/rooteq/ros2_ws/install/quadro/share/quadro/des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; visual mesh filename=file:///home/rooteq/ros2_ws/install/quadro/share/quadro/des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
- link back_plate: geometry collision mesh filename=file:///home/rooteq/ros2_ws/install/quadro/share/quadro/des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; visual mesh filename=file:///home/rooteq/ros2_ws/install/quadro/share/quadro/des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
- link l4_l: mass 0.0940232 -> 0.0817713; geometry collision mesh filename=file:///home/rooteq/ros2_ws/install/quadro/share/quadro/des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; visual mesh filename=file:///home/rooteq/ros2_ws/install/quadro/share/quadro/des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
- link l4_l_2: mass 0.0940232 -> 0.0817713; geometry collision mesh filename=file:///home/rooteq/ros2_ws/install/quadro/share/quadro/des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; visual mesh filename=file:///home/rooteq/ros2_ws/install/quadro/share/quadro/des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
- link l4_r: mass 0.0940232 -> 0.0817713; geometry collision mesh filename=file:///home/rooteq/ros2_ws/install/quadro/share/quadro/des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; visual mesh filename=file:///home/rooteq/ros2_ws/install/quadro/share/quadro/des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
- link l4_r_2: mass 0.0940232 -> 0.0817713; geometry collision mesh filename=file:///home/rooteq/ros2_ws/install/quadro/share/quadro/des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; visual mesh filename=file:///home/rooteq/ros2_ws/install/quadro/share/quadro/des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
- link motor: geometry collision mesh filename=file:///home/rooteq/ros2_ws/install/quadro/share/quadro/des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; visual mesh filename=file:///home/rooteq/ros2_ws/install/quadro/share/quadro/des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
- link motor_2: geometry collision mesh filename=file:///home/rooteq/ros2_ws/install/quadro/share/quadro/des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; visual mesh filename=file:///home/rooteq/ros2_ws/install/quadro/share/quadro/des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
- link shaft: geometry collision mesh filename=file:///home/rooteq/ros2_ws/install/quadro/share/quadro/des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; visual mesh filename=file:///home/rooteq/ros2_ws/install/quadro/share/quadro/des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
- link shaft_10: geometry collision mesh filename=file:///home/rooteq/ros2_ws/install/quadro/share/quadro/des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; visual mesh filename=file:///home/rooteq/ros2_ws/install/quadro/share/quadro/des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
- link shaft_2: geometry collision mesh filename=file:///home/rooteq/ros2_ws/install/quadro/share/quadro/des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; visual mesh filename=file:///home/rooteq/ros2_ws/install/quadro/share/quadro/des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
- link shaft_3: geometry collision mesh filename=file:///home/rooteq/ros2_ws/install/quadro/share/quadro/des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; visual mesh filename=file:///home/rooteq/ros2_ws/install/quadro/share/quadro/des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
- link shaft_4: geometry collision mesh filename=file:///home/rooteq/ros2_ws/install/quadro/share/quadro/des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; visual mesh filename=file:///home/rooteq/ros2_ws/install/quadro/share/quadro/des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
- link shaft_5: geometry collision mesh filename=file:///home/rooteq/ros2_ws/install/quadro/share/quadro/des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; visual mesh filename=file:///home/rooteq/ros2_ws/install/quadro/share/quadro/des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
- link shaft_6: geometry collision mesh filename=file:///home/rooteq/ros2_ws/install/quadro/share/quadro/des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; visual mesh filename=file:///home/rooteq/ros2_ws/install/quadro/share/quadro/des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
- link shaft_7: geometry collision mesh filename=file:///home/rooteq/ros2_ws/install/quadro/share/quadro/des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; visual mesh filename=file:///home/rooteq/ros2_ws/install/quadro/share/quadro/des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
- link shaft_8: geometry collision mesh filename=file:///home/rooteq/ros2_ws/install/quadro/share/quadro/des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; visual mesh filename=file:///home/rooteq/ros2_ws/install/quadro/share/quadro/des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
- link shaft_9: geometry collision mesh filename=file:///home/rooteq/ros2_ws/install/quadro/share/quadro/des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; visual mesh filename=file:///home/rooteq/ros2_ws/install/quadro/share/quadro/des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
Joints:
- removed joint bl_foot_frame
- removed joint br_foot_frame
- removed joint fl_foot_frame
- removed joint fr_foot_frame
- added joint bl_feet: type fixed, parent l4_l, child feet_2, origin xyz=-0 0.163 -0.004 rpy=-1.5708 -0 -3.14159, axis 0 0 1, limit lower=-3.14 upper=3.14 effort=10 velocity=12
- added joint br_feet: type fixed, parent l4_r, child feet, origin xyz=0 -0.163 -0.004 rpy=-1.5708 -0 -0, axis 0 0 1, limit lower=-3.14 upper=3.14 effort=10 velocity=12
- added joint fl_feet: type fixed, parent l4_l_2, child feet_4, origin xyz=0 0.163 -0.004 rpy=-1.5708 0 3.14159, axis 0 0 1, limit lower=-3.14 upper=3.14 effort=10 velocity=12
- added joint fr_feet: type fixed, parent l4_r_2, child feet_3, origin xyz=-0 -0.163 -0.004 rpy=-1.5708 0 0, axis 0 0 1, limit lower=-3.14 upper=3.14 effort=10 velocity=12
- joint bl_l4_l3: origin xyz=0.129917 0.0934105 -0.0735 rpy=-1.63758e-14 6.77236e-15 1.53589 -> xyz=0.129917 0.0934105 -0.0735 rpy=-0 0 1.53589
- joint bl_m1_s1: origin xyz=-0.0840337 0.126935 -0.00844105 rpy=-1.5708 -9.60008e-14 -3.14159 -> xyz=0.0549617 0.114632 7.33841e-06 rpy=-1.5708 -0 -3.14159
- joint bl_m3_s3: origin xyz=7.21645e-16 -1.52656e-16 -0.0495 rpy=1.21014e-14 5.23193e-15 -2.3911 -> xyz=-0 0 -0.0495 rpy=-0 -0 -2.3911
- joint br_l4_l3: origin xyz=0.159217 -0.0159373 -0.0735 rpy=-1.72085e-15 4.38538e-15 -1.01229 -> xyz=0.159217 -0.0159373 -0.0735 rpy=-0 0 -1.01229
- joint br_m1_s1: origin xyz=-0.194034 0.126935 -0.00844105 rpy=-1.5708 -8.11125e-15 3.14159 -> xyz=-0.0550383 0.114632 7.33851e-06 rpy=-1.5708 -0 3.14159
- joint br_m3_s3: origin xyz=2.77556e-17 -2.77556e-17 -0.0495 rpy=-6.10623e-16 8.46545e-16 -0.226893 -> xyz=0 -0 -0.0495 rpy=-0 0 -0.226893
- joint fl_l4_l3: origin xyz=-0.159217 -0.0159373 -0.0735 rpy=1.16573e-15 -4.996e-16 -2.1293 -> xyz=-0.159217 -0.0159373 -0.0735 rpy=0 -0 -2.1293
- joint fl_m1_s1: origin xyz=-0.0840337 -0.102065 -0.00844105 rpy=1.5708 -0 -3.14159 -> xyz=0.0549617 -0.114368 7.33841e-06 rpy=1.5708 -0 -3.14159
- joint fl_m3_s3: origin xyz=0 0 -0.0495 rpy=-1.55431e-15 2.77556e-17 0.226893 -> xyz=0 0 -0.0495 rpy=-0 0 0.226893
- joint fr_l4_l3: origin xyz=0.159217 -0.0159373 -0.0735 rpy=1.38778e-15 -2.77556e-16 -1.01229 -> xyz=0.159217 -0.0159373 -0.0735 rpy=0 -0 -1.01229
- joint fr_m1_s1: origin xyz=-0.194034 -0.102065 -0.00844105 rpy=1.5708 -0 -3.14159 -> xyz=-0.0550383 -0.114368 7.33851e-06 rpy=1.5708 -0 -3.14159
- joint fr_m3_s3: origin xyz=0 -2.77556e-17 -0.0495 rpy=-1.11022e-15 -1.11022e-15 -0.226893 -> xyz=0 -0 -0.0495 rpy=-0 -0 -0.226893

File: isaac_sim_files/quadro.xacro (robot description, xacro)
@@ -4,280 +4,25 @@
 <xacro:include filename="$(find quadro)/description/materials.xacro" />
 <!-- <xacro:include filename="$(find quadro)/description/quadro.trans" /> -->
+  <!-- Link back_plate -->
   <link name="back_plate">
     <inertial>
-      <origin xyz="-0.139034 0.00733582 -0.013731" rpy="0 0 0"/>
+      <origin xyz="-3.82601e-05 -0.00496654 -0.00528261" rpy="0 0 0"/>
       <mass value="2.59053"/>
-      <inertia ixx="0.0255846" ixy="-4.15339e-05" ixz="-1.35405e-12" iyy="0.00872593" iyz="-0.000207516" izz="0.0313278"/>
-    </inertial>
-    <!-- Part back_stop -->
-    <visual>
-      <origin xyz="-0.139034 -0.0331652 -0.058441" rpy="0 -0 0"/>
-      <geometry>
-        <mesh filename="file://$(find quadro)/description/assets/back_stop.stl"/>
-      </geometry>
-      <material name="back_stop_material">
-        <color rgba="1 0.756863 0.054902 1"/>
-      </material>
-    </visual>
-    <collision>
-      <origin xyz="-0.139034 -0.0331652 -0.058441" rpy="0 -0 0"/>
-      <geometry>
-        <mesh filename="file://$(find quadro)/description/assets/back_stop.stl"/>
-      </geometry>
-    </collision>
-    <!-- Part side_pipe -->
-    <visual>
-      <origin xyz="-0.286981 0.105935 -0.058441" rpy="0 -0 0"/>
-      <geometry>
-        <mesh filename="file://$(find quadro)/description/assets/side_pipe.stl"/>
-      </geometry>
-      <material name="side_pipe_material">
-        <color rgba="0 0 0 1"/>
-      </material>
-    </visual>
-    <collision>
-      <origin xyz="-0.286981 0.105935 -0.058441" rpy="0 -0 0"/>
-      <geometry>
-        <mesh filename="file://$(find quadro)/description/assets/side_pipe.stl"/>
-      </geometry>
-    </collision>
-    <!-- Part side_cover -->
-    <visual>
-      <origin xyz="-0.139034 -0.0810652 -0.058441" rpy="2.4928e-28 -8.23912e-18 -3.14159"/>
-      <geometry>
-        <mesh filename="file://$(find quadro)/description/assets/side_cover.stl"/>
-      </geometry>
-      <material name="side_cover_material">
-        <color rgba="0.647059 0.647059 0.647059 1"/>
-      </material>
-    </visual>
-    <collision>
-      <origin xyz="-0.139034 -0.0810652 -0.058441" rpy="2.4928e-28 -8.23912e-18 -3.14159"/>
-      <geometry>
-        <mesh filename="file://$(find quadro)/description/assets/side_cover.stl"/>
-      </geometry>
-    </collision>
-    <!-- Part back_plate -->
-    <visual>
-      <origin xyz="-0.139034 0.105935 -0.058441" rpy="-3.9443e-31 6.56859e-46 -1.79651e-46"/>
-      <geometry>
-        <mesh filename="file://$(find quadro)/description/assets/back_plate.stl"/>
-      </geometry>
-      <material name="back_plate_material">
-        <color rgba="1 0.756863 0.054902 1"/>
-      </material>
-    </visual>
-    <collision>
-      <origin xyz="-0.139034 0.105935 -0.058441" rpy="-3.9443e-31 6.56859e-46 -1.79651e-46"/>
-      <geometry>
-        <mesh filename="file://$(find quadro)/description/assets/back_plate.stl"/>
-      </geometry>
-    </collision>
-    <!-- Part battery -->
-    <visual>
-      <origin xyz="-0.0725337 -0.0315652 -0.029441" rpy="0 -6.12323e-17 1.5708"/>
-      <geometry>
-        <mesh filename="file://$(find quadro)/description/assets/battery.stl"/>
-      </geometry>
-      <material name="battery_material">
-        <color rgba="0.768627 0.886275 0.952941 1"/>
-      </material>
-    </visual>
-    <collision>
-      <origin xyz="-0.0725337 -0.0315652 -0.029441" rpy="0 -6.12323e-17 1.5708"/>
-      <geometry>
-        <mesh filename="file://$(find quadro)/description/assets/battery.stl"/>
-      </geometry>
-    </collision>
-    <!-- Part motor -->
-    <visual>
-      <origin xyz="-0.194034 -0.0920652 -0.00844105" rpy="3.14159 5.95406e-36 -1.5708"/>
-      <geometry>
-        <mesh filename="file://$(find quadro)/description/assets/motor.stl"/>
-      </geometry>
-      <material name="motor_material">
-        <color rgba="0.498039 0.498039 0.498039 1"/>
-      </material>
-    </visual>
-    <collision>
-      <origin xyz="-0.194034 -0.0920652 -0.00844105" rpy="3.14159 5.95406e-36 -1.5708"/>
-      <geometry>
-        <mesh filename="file://$(find quadro)/description/assets/motor.stl"/>
-      </geometry>
-    </collision>
-    <!-- Part side_cover_2 -->
-    <visual>
-      <origin xyz="-0.139034 0.105935 -0.058441" rpy="0 -8.23912e-18 2.00179e-32"/>
-      <geometry>
-        <mesh filename="file://$(find quadro)/description/assets/side_cover.stl"/>
-      </geometry>
-      <material name="side_cover_2_material">
-        <color rgba="0.647059 0.647059 0.647059 1"/>
-      </material>
-    </visual>
-    <collision>
-      <origin xyz="-0.139034 0.105935 -0.058441" rpy="0 -8.23912e-18 2.00179e-32"/>
-      <geometry>
-        <mesh filename="file://$(find quadro)/description/assets/side_cover.stl"/>
-      </geometry>
-    </collision>
-    <!-- Part motor_2 -->
-    <visual>
-      <origin xyz="-0.194034 0.116935 -0.00844105" rpy="-3.14159 7.88861e-31 1.5708"/>
-      <geometry>
-        <mesh filename="file://$(find quadro)/description/assets/motor.stl"/>
-      </geometry>
-      <material name="motor_2_material">
-        <color rgba="0.498039 0.498039 0.498039 1"/>
-      </material>
-    </visual>
-    <collision>
-      <origin xyz="-0.194034 0.116935 -0.00844105" rpy="-3.14159 7.88861e-31 1.5708"/>
-      <geometry>
-        <mesh filename="file://$(find quadro)/description/assets/motor.stl"/>
-      </geometry>
-    </collision>
-    <!-- Part motor_3 -->
-    <visual>
-      <origin xyz="-0.0840337 -0.0920652 -0.00844105" rpy="3.14159 5.95406e-36 -1.5708"/>
-      <geometry>
-        <mesh filename="file://$(find quadro)/description/assets/motor.stl"/>
-      </geometry>
-      <material name="motor_3_material">
-        <color rgba="0.498039 0.498039 0.498039 1"/>
-      </material>
-    </visual>
-    <collision>
-      <origin xyz="-0.0840337 -0.0920652 -0.00844105" rpy="3.14159 5.95406e-36 -1.5708"/>
-      <geometry>
-        <mesh filename="file://$(find quadro)/description/assets/motor.stl"/>
-      </geometry>
-    </collision>
-    <!-- Part bot_pipe_half -->
-    <visual>
-      <origin xyz="-0.139034 0.439935 -0.058441" rpy="3.14159 -0 0"/>
-      <geometry>
-        <mesh filename="file://$(find quadro)/description/assets/bot_pipe_half.stl"/>
-      </geometry>
-      <material name="bot_pipe_half_material">
-        <color rgba="0.972549 0.529412 0.00392157 1"/>
-      </material>
-    </visual>
-    <collision>
-      <origin xyz="-0.139034 0.439935 -0.058441" rpy="3.14159 -0 0"/>
-      <geometry>
-        <mesh filename="file://$(find quadro)/description/assets/bot_pipe_half.stl"/>
-      </geometry>
-    </collision>
-    <!-- Part side_pipe_2 -->
-    <visual>
-      <origin xyz="-0.139034 -0.0810652 0.095559" rpy="3.14159 -0 0"/>
-      <geometry>
-        <mesh filename="file://$(find quadro)/description/assets/side_pipe.stl"/>
-      </geometry>
-      <material name="side_pipe_2_material">
-        <color rgba="0 0 0 1"/>
-      </material>
-    </visual>
-    <collision>
-      <origin xyz="-0.139034 -0.0810652 0.095559" rpy="3.14159 -0 0"/>
-      <geometry>
-        <mesh filename="file://$(find quadro)/description/assets/side_pipe.stl"/>
-      </geometry>
-    </collision>
-    <!-- Part motor_4 -->
-    <visual>
-      <origin xyz="-0.0840337 0.116935 -0.00844105" rpy="-3.14159 7.88861e-31 1.5708"/>
-      <geometry>
-        <mesh filename="file://$(find quadro)/description/assets/motor.stl"/>
-      </geometry>
-      <material name="motor_4_material">
-        <color rgba="0.498039 0.498039 0.498039 1"/>
-      </material>
-    </visual>
-    <collision>
-      <origin xyz="-0.0840337 0.116935 -0.00844105" rpy="-3.14159 7.88861e-31 1.5708"/>
-      <geometry>
-        <mesh filename="file://$(find quadro)/description/assets/motor.stl"/>
-      </geometry>
-    </collision>
-    <!-- Part back_stop_2 -->
-    <visual>
-      <origin xyz="-0.139034 0.0580348 -0.058441" rpy="0 -0 -3.14159"/>
-      <geometry>
-        <mesh filename="file://$(find quadro)/description/assets/back_stop.stl"/>
-      </geometry>
-      <material name="back_stop_2_material">
-        <color rgba="1 0.756863 0.054902 1"/>
-      </material>
-    </visual>
-    <collision>
-      <origin xyz="-0.139034 0.0580348 -0.058441" rpy="0 -0 -3.14159"/>
-      <geometry>
-        <mesh filename="file://$(find quadro)/description/assets/back_stop.stl"/>
-      </geometry>
-    </collision>
-    <!-- Part back_plate_2 -->
-    <visual>
-      <origin xyz="-0.139034 -0.0810652 -0.058441" rpy="0 -0 3.14159"/>
-      <geometry>
-        <mesh filename="file://$(find quadro)/description/assets/back_plate.stl"/>
-      </geometry>
-      <material name="back_plate_2_material">
-        <color rgba="1 0.756863 0.054902 1"/>
-      </material>
-    </visual>
-    <collision>
-      <origin xyz="-0.139034 -0.0810652 -0.058441" rpy="0 -0 3.14159"/>
-      <geometry>
-        <mesh filename="file://$(find quadro)/description/assets/back_plate.stl"/>
-      </geometry>
-    </collision>
-    <!-- Part bot_pipe_half_2 -->
-    <visual>
-      <origin xyz="-0.139034 -0.415065 -0.058441" rpy="0 -0 0"/>
-      <geometry>
-        <mesh filename="file://$(find quadro)/description/assets/bot_pipe_half.stl"/>
-      </geometry>
-      <material name="bot_pipe_half_2_material">
-        <color rgba="0.972549 0.529412 0.00392157 1"/>
-      </material>
-    </visual>
-    <collision>
-      <origin xyz="-0.139034 -0.415065 -0.058441" rpy="0 -0 0"/>
-      <geometry>
-        <mesh filename="file://$(find quadro)/description/assets/bot_pipe_half.stl"/>
-      </geometry>
-    </collision>
-    <!-- Part mid_clamp -->
-    <visual>
-      <origin xyz="-0.139034 0.245535 -0.058441" rpy="0 -0 0"/>
-      <geometry>
-        <mesh filename="file://$(find quadro)/description/assets/mid_clamp.stl"/>
-      </geometry>
-      <material name="mid_clamp_material">
-        <color rgba="1 0.756863 0.054902 1"/>
-      </material>
-    </visual>
-    <collision>
-      <origin xyz="-0.139034 0.245535 -0.058441" rpy="0 -0 0"/>
-      <geometry>
-        <mesh filename="file://$(find quadro)/description/assets/mid_clamp.stl"/>
-      </geometry>
-    </collision>
-    <!-- Part battery_2 -->
-    <visual>
-      <origin xyz="-0.205534 -0.0315652 -0.029441" rpy="3.14159 -0 1.5708"/>
-      <geometry>
-        <mesh filename="file://$(find quadro)/description/assets/battery.stl"/>
-      </geometry>
-      <material name="battery_2_material">
-        <color rgba="0.768627 0.886275 0.952941 1"/>
-      </material>
-    </visual>
-    <collision>
-      <origin xyz="-0.205534 -0.0315652 -0.029441" rpy="3.14159 -0 1.5708"/>
-      <geometry>
-        <mesh filename="file://$(find quadro)/description/assets/battery.stl"/>
+      <inertia ixx="0.0255846" ixy="-4.15339e-05" ixz="4e-12" iyy="0.00872593" iyz="-0.000207516" izz="0.0313278"/>
+    </inertial>
+    <!-- Part back_plate_parts -->
+    <visual>
+      <origin xyz="-3.82601e-05 -0.00496654 -0.00528261" rpy="0 -0 0"/>
+      <geometry>
+        <mesh filename="file://$(find quadro)/descritpion/assets/merged/back_plate_visual.stl"/>
+      </geometry>
+      <material name="back_plate_parts_material">
+        <color rgba="0.67735 0.643034 0.48069 1"/>
+      </material>
+    </visual>
+    <collision>
+      <origin xyz="-3.82601e-05 -0.00496654 -0.00528261" rpy="0 -0 0"/>
+      <geometry>
+        <mesh filename="file://$(find quadro)/descritpion/assets/merged/back_plate_collision.stl"/>
       </geometry>
     </collision>
@@ -290,50 +35,18 @@
       <inertia ixx="0.000550761" ixy="-6.00381e-05" ixz="-1.13918e-05" iyy="0.00055728" iyz="1.18589e-05" izz="0.000239291"/>
     </inertial>
-    <!-- Part lin_1_support_br -->
-    <visual>
-      <origin xyz="-0.019799 0.019799 -0.0735" rpy="0.785398 -1.5708 0"/>
-      <geometry>
-        <mesh filename="file://$(find quadro)/description/assets/lin_1_support_br.stl"/>
-      </geometry>
-      <material name="lin_1_support_br_material">
-        <color rgba="0.901961 0.901961 0.901961 1"/>
-      </material>
-    </visual>
-    <collision>
-      <origin xyz="-0.019799 0.019799 -0.0735" rpy="0.785398 -1.5708 0"/>
-      <geometry>
-        <mesh filename="file://$(find quadro)/description/assets/lin_1_support_br.stl"/>
-      </geometry>
-    </collision>
-    <!-- Part motor_5 -->
-    <visual>
-      <origin xyz="-0.0120208 0.0120208 -0.0735" rpy="-1.5708 4.94218e-17 -0.785398"/>
-      <geometry>
-        <mesh filename="file://$(find quadro)/description/assets/motor.stl"/>
-      </geometry>
-      <material name="motor_5_material">
-        <color rgba="0.498039 0.498039 0.498039 1"/>
-      </material>
-    </visual>
-    <collision>
-      <origin xyz="-0.0120208 0.0120208 -0.0735" rpy="-1.5708 4.94218e-17 -0.785398"/>
-      <geometry>
-        <mesh filename="file://$(find quadro)/description/assets/motor.stl"/>
-      </geometry>
-    </collision>
-    <!-- Part shaft -->
-    <visual>
-      <origin xyz="0 0 0.01" rpy="1.5708 1.5708 0"/>
-      <geometry>
-        <mesh filename="file://$(find quadro)/description/assets/shaft.stl"/>
-      </geometry>
-      <material name="shaft_material">
-        <color rgba="0.498039 0.498039 0.498039 1"/>
-      </material>
-    </visual>
-    <collision>
-      <origin xyz="0 0 0.01" rpy="1.5708 1.5708 0"/>
-      <geometry>
-        <mesh filename="file://$(find quadro)/description/assets/shaft.stl"/>
+    <!-- Part shaft_parts -->
+    <visual>
+      <origin xyz="-0.00474046 0.00407901 -0.0612986" rpy="-1.5708 0 -3.14159"/>
+      <geometry>
+        <mesh filename="file://$(find quadro)/descritpion/assets/merged/shaft_visual.stl"/>
+      </geometry>
+      <material name="shaft_parts_material">
+        <color rgba="0.556109 0.556109 0.556109 1"/>
+      </material>
+    </visual>
+    <collision>
+      <origin xyz="-0.00474046 0.00407901 -0.0612986" rpy="-1.5708 0 -3.14159"/>
+      <geometry>
+        <mesh filename="file://$(find quadro)/descritpion/assets/merged/shaft_collision.stl"/>
       </geometry>
     </collision>
@@ -346,82 +59,18 @@
       <inertia ixx="0.000439148" ixy="6.14395e-05" ixz="0.000140002" iyy="0.000912333" iyz="-3.78102e-05" izz="0.000883052"/>
     </inertial>
-    <!-- Part bot_r -->
-    <visual>
-      <origin xyz="5.55112e-16 3.60822e-16 0.1275" rpy="-1.5708 1.35308e-15 -0.0872665"/>
-      <geometry>
-        <mesh filename="file://$(find quadro)/description/assets/bot_r.stl"/>
-      </geometry>
-      <material name="bot_r_material">
-        <color rgba="0.901961 0.901961 0.901961 1"/>
-      </material>
-    </visual>
-    <collision>
-      <origin xyz="5.55112e-16 3.60822e-16 0.1275" rpy="-1.5708 1.35308e-15 -0.0872665"/>
-      <geometry>
-        <mesh filename="file://$(find quadro)/description/assets/bot_r.stl"/>
-      </geometry>
-    </collision>
-    <!-- Part top_r -->
-    <visual>
-      <origin xyz="4.71845e-16 3.88578e-16 0.1275" rpy="-1.5708 1.20043e-15 -0.0872665"/>
-      <geometry>
-        <mesh filename="file://$(find quadro)/description/assets/top_r.stl"/>
-      </geometry>
-      <material name="top_r_material">
-        <color rgba="0.901961 0.901961 0.901961 1"/>
-      </material>
-    </visual>
-    <collision>
-      <origin xyz="4.71845e-16 3.88578e-16 0.1275" rpy="-1.5708 1.20043e-15 -0.0872665"/>
-      <geometry>
-        <mesh filename="file://$(find quadro)/description/assets/top_r.stl"/>
-      </geometry>
-    </collision>
-    <!-- Part shaft_2 -->
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